File: nonSNES.kicad_sch (KiCad schematic)
At the start: 9 parts, among them J1 Jack-DC, P3 Conn_01x02_Male, T1 L_Coupled, U1 CPU, U12 L7805

Commit message: add ram and voltage reg
Parts:
- added C34: 0.1uF, Capacitor_SMD:C_0805_2012Metric, symbol Device:C
- added C81: 1uF, Capacitor_SMD:C_0805_2012Metric, symbol Device:C
- added U4, U5: KM62256CLP, Package_SO:SOIC-28W_7.5x17.9mm_P1.27mm, symbol Memory_RAM:KM62256CLP
- J1: footprint Connector_Molex:Molex_Mega-Fit_76829-0102_2x01_P5.70mm_Vertical -> SNES_Library:DcJack
Connections:
- net GNDPWR: now also U12.2 (GND), C34.2, C81.2
- net at P3.2 (Pin_2), U12.1 (IN): now also C34.1
- net VCC: now reaches U12.3 (OUT)
- net VCC: now also C81.1

Commit message: connect vram data lines
Parts:
- added C93: C, Capacitor_SMD:C_0805_2012Metric, symbol Device:C
- added C95, C97: 0.1uF, Capacitor_SMD:C_0805_2012Metric, symbol Device:C
- added P1: CASSETTE, Connector_DIN:DIN41612_R_2x32_Male_Vertical_THT, symbol SNES_Library:CASSETTE
- U4, U5: value KM62256CLP -> MS62256CL-10FC
Connections:
- net GNDPWR: now also U4.14 (GND), U4.20 (~{CS}), U5.14 (GND), U5.20 (~{CS}), C93.2, C95.2, C97.2
- net VCC: now also U1.1 (VCC), U1.34 (VCC), U4.28 (VCC), U5.28 (VCC), C93.1, C95.1, C97.1
- net D0: now reaches U5.11 (Q0)
- net D0: now also U4.11 (Q0)
- net D1: now reaches U5.12 (Q1)
- net D1: now also U4.12 (Q1)
- net D2: now reaches U5.13 (Q2)
- net D2: now also U4.13 (Q2)
- net D3: now reaches U5.15 (Q3)
- net D3: now also U4.15 (Q3)
- net D4: now reaches U5.16 (Q4)
- net D4: now also U4.16 (Q4)
- net D5: now reaches U5.17 (Q5)
- net D5: now also U4.17 (Q5)
- net D6: now reaches U5.18 (Q6)
- net D6: now also U4.18 (Q6)
- net D7: now reaches U5.19 (Q7)
- net D7: now also U4.19 (Q7)

Commit message: add ppu
Parts:
- added U?: PPU2, symbol SNES_Library:PPU2
- added U?: PPU1, symbol SNES_Library:PPU1

Commit message: fix misaligned pins
Parts:
- added C92, C94: C, Capacitor_SMD:C_0805_2012Metric, symbol Device:C
- U2, U3: renamed from U?; footprint (none) -> Package_QFP:PQFP-100_14x20mm_P0.65mm
- U4, U5: footprint Package_SO:SOIC-28W_7.5x17.9mm_P1.27mm -> Package_DIP:DIP-28_W15.24mm
Connections:
- net GNDPWR: now also C92.2, C94.2
- net VCC: now also U1.59 (VCC), U1.85 (VCC), U2.13 (VCC), U2.36 (VCC), U2.62 (VCC), U2.81 (VCC), U3.32 (VCC), U3.5 (VCC), U3.59 (VCC), U3.83 (VCC), C92.1, C94.1

Commit message: fix ram package
Parts:
- U4, U5: footprint Package_DIP:DIP-28_W15.24mm -> Package_SO:SOIC-28W_7.5x17.9mm_P1.27mm
Changed lines of the file:
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@@
       (effects (font (size 1.27 1.27)) (justify left))
     )
-    (property "Footprint" "Package_DIP:DIP-28_W15.24mm" (id 2) (at 165.1 78.74 0)
+    (property "Footprint" "Package_SO:SOIC-28W_7.5x17.9mm_P1.27mm" (id 2) (at 165.1 78.74 0)
       (effects (font (size 1.27 1.27)) hide)
     )
@@
       (effects (font (size 1.27 1.27)) (justify left))
     )
-    (property "Footprint" "Package_DIP:DIP-28_W15.24mm" (id 2) (at 165.1 135.89 0)
+    (property "Footprint" "Package_SO:SOIC-28W_7.5x17.9mm_P1.27mm" (id 2) (at 165.1 135.89 0)
       (effects (font (size 1.27 1.27)) hide)
     )
@@
     )
     (path "/c1bcc54b-122a-4641-a51e-ce59f13fb71d"
-      (reference "U4") (unit 1) (value "MS62256CL-10FC") (footprint "Package_DIP:DIP-28_W15.24mm")
+      (reference "U4") (unit 1) (value "MS62256CL-10FC") (footprint "Package_SO:SOIC-28W_7.5x17.9mm_P1.27mm")
     )
     (path "/ec9b8000-6dbd-41b7-bfe9-8eb43218a4f1"
-      (reference "U5") (unit 1) (value "MS62256CL-10FC") (footprint "Package_DIP:DIP-28_W15.24mm")
+      (reference "U5") (unit 1) (value "MS62256CL-10FC") (footprint "Package_SO:SOIC-28W_7.5x17.9mm_P1.27mm")
     )
     (path "/080a219d-424b-44f8-92f5-004ac6a80de0"

Commit message: add crystal
Parts:
- added X1: Crystal, symbol Device:Crystal

Commit message: add controller port
Parts:
- added C107: 0.01u, Capacitor_SMD:C_0805_2012Metric, symbol Device:C_Polarized
- added C35, C36, C37, C38, C39, C40, C41, C42, C43: 330p, Capacitor_SMD:C_0805_2012Metric, symbol Device:C_Polarized
- added DA10, DA2, DA3, DA4, DA5, DA7, DA8, DA9: D, Package_TO_SOT_SMD:SOT-23, symbol Device:D
- added P2: Conn_2Rows-11Pins, Connector_JST:JST_ZE_B11B-ZESK-D_1x11_P1.50mm_Vertical, symbol Connector_Generic:Conn_2Rows-11Pins
- added R78, R80, R82: 10k, Resistor_SMD:R_0805_2012Metric, symbol Device:R
- added R83, R84, R85, R86, R87, R88, R89, R90, R91: 100, Resistor_SMD:R_0805_2012Metric, symbol Device:R
- X1: footprint (none) -> Crystal:Crystal_HC49-4H_Vertical
Connections:
- net VCC: now also U3.94 (AVCC), C107.1, DA10.1 (K), DA7.1 (K), DA8.1 (K), DA9.1 (K), P2.1 (Pin_1), R78.1, R80.1, R82.1
- net GND: now reaches U3.16 (GND)
- net GND: now also P1.SHIELD (GND), U1.18 (GND), U1.47 (GND), U1.79 (GND), U1.90 (GND), U2.22 (GND), U2.45 (GND), U2.77 (GND), U2.96 (GND), U3.30 (PALMODE), U3.35 (GND), U3.68 (GND), U3.90 (TST12), U3.91 (TST13), U3.92 (TST14), U3.93 (TST15), U3.99 (GND), C107.2, C35.2, C36.2, C37.2, C38.2, C39.2, C40.2, C41.2, C42.2, C43.2, DA2.2 (A), DA3.2 (A), DA4.2 (A), DA5.2 (A), P2.11 (Pin_11)
- net VDB0: now reaches U3.51 (VDB0)
- net VDB0: now also U2.28 (VDB0), U3.69 (EXT0), U4.11 (Q0)
- net VDB1: now reaches U3.52 (VDB1)
- net VDB1: now also U2.29 (VDB1), U3.70 (EXT1), U4.12 (Q1)
- net VDB2: now reaches U3.53 (VDB2)
- net VDB2: now also U2.30 (VDB2), U3.71 (EXT2), U4.13 (Q2)
- net VDB3: now reaches U3.54 (VDB3)
- net VDB3: now also U2.31 (VDB3), U3.72 (EXT3), U4.15 (Q3)
- net VDB4: now reaches U3.55 (VDB4)
- net VDB4: now also U2.32 (VDB4), U3.73 (EXT4), U4.16 (Q4)
- net VDB5: now reaches U3.56 (VDB5)
- net VDB5: now also U2.33 (VDB5), U3.74 (EXT5), U4.17 (Q5)
- net VDB6: now reaches U3.57 (VDB6)
- net VDB6: now also U2.34 (VDB6), U3.75 (EXT6), U4.18 (Q6)
- net VDB7: now reaches U3.58 (VDB7)
- net VDB7: now also U2.35 (VDB7), U3.76 (EXT7), U4.19 (Q7)
- net VDA0: now reaches U3.60 (VDA0)
- net VDA0: now also U2.37 (VDA0), U5.11 (Q0)
- net VDA1: now reaches U3.61 (VDA1)
- net VDA1: now also U2.38 (VDA1), U5.12 (Q1)
- net VDA2: now reaches U3.62 (VDA2)
- net VDA2: now also U2.39 (VDA2), U5.13 (Q2)
- net VDA3: now reaches U3.63 (VDA3)
- net VDA3: now also U2.40 (VDA3), U5.15 (Q3)
- net VDA4: now reaches U3.64 (VDA4)
- net VDA4: now also U2.41 (VDA4), U5.16 (Q4)
- net VDA5: now reaches U3.65 (VDA5)
- net VDA5: now also U2.42 (VDA5), U5.17 (Q5)
- net VDA6: now reaches U3.66 (VDA6)
- net VDA6: now also U2.43 (VDA6), U5.18 (Q6)
- net VDA7: now reaches U3.67 (VDA7)
- net VDA7: now also U2.44 (VDA7), U5.19 (Q7)
- net VA14: now reaches U2.47 (VA14)
- net VA14: now also U4.1 (A14), U5.1 (A14)
- net VAB13: now reaches U2.48 (VAB13)
- net VAB13: now also U4.26 (A13)
- net VAB12: now reaches U2.49 (VAB12)
- net VAB12: now also U4.2 (A12)
- net VAB11: now reaches U2.50 (VAB11)
- net VAB11: now also U4.23 (A11)
- net VAB10: now reaches U2.51 (VAB10)
- net VAB10: now also U4.21 (A10)
- net VAB9: now reaches U2.52 (VAB9)
- net VAB9: now also U4.24 (A9)
- net VAB8: now reaches U2.53 (VAB8)
- net VAB8: now also U4.25 (A8)
- net VAB7: now reaches U2.54 (VAB7)
- net VAB7: now also U4.3 (A7)
- net VAB6: now reaches U2.55 (VAB6)
- net VAB6: now also U4.4 (A6)
- net VAB5: now reaches U2.56 (VAB5)
- net VAB5: now also U4.5 (A5)
- net VAB4: now reaches U2.57 (VAB4)
- net VAB4: now also U4.6 (A4)
- net VAB3: now reaches U2.58 (VAB3)
- net VAB3: now also U4.7 (A3)
- net VAB2: now reaches U2.59 (VAB2)
- net VAB2: now also U4.8 (A2)
- net VAB1: now reaches U2.60 (VAB1)
- net VAB1: now also U4.9 (A1)
- net VAB0: now reaches U2.61 (VAB0)
- net VAB0: now also U4.10 (A0)
- net VAA13: now reaches U2.63 (VAA13)
- net VAA13: now also U5.26 (A13)
- net VAA12: now reaches U2.64 (VAA12)
- net VAA12: now also U5.2 (A12)
- net VAA11: now reaches U2.65 (VAA11)
- net VAA11: now also U5.23 (A11)
- net VAA10: now reaches U2.66 (VAA10)
- net VAA10: now also U5.21 (A10)
- net VAA9: now reaches U2.67 (VAA9)
- net VAA9: now also U5.24 (A9)
- net VAA8: now reaches U2.68 (VAA8)
- net VAA8: now also U5.25 (A8)
- net VAA7: now reaches U2.69 (VAA7)
- net VAA7: now also U5.3 (A7)
- net VAA6: now reaches U2.70 (VAA6)
- net VAA6: now also U5.4 (A6)
- net VAA5: now reaches U2.71 (VAA5)
- net VAA5: now also U5.5 (A5)
- net VAA4: now reaches U2.72 (VAA4)
- net VAA4: now also U5.6 (A4)
- net VAA3: now reaches U2.73 (VAA3)
- net VAA3: now also U5.7 (A3)
- net VAA2: now reaches U2.74 (VAA2)
- net VAA2: now also U5.8 (A2)
- net VAA1: now reaches U2.75 (VAA1)
- net VAA1: now also U5.9 (A1)
- net VAA0: now reaches U2.76 (VAA0)
- net VAA0: now also U5.10 (A0)
- removed net D0: U4.11 (Q0), U5.11 (Q0)
- removed net D1: U4.12 (Q1), U5.12 (Q1)
- removed net D2: U4.13 (Q2), U5.13 (Q2)
- removed net D3: U4.15 (Q3), U5.15 (Q3)
- removed net D4: U4.16 (Q4), U5.16 (Q4)
- removed net D5: U4.17 (Q5), U5.17 (Q5)
- removed net D6: U4.18 (Q6), U5.18 (Q6)
- removed net D7: U4.19 (Q7), U5.19 (Q7)
- new net: C42.1, P2.9 (Pin_9), R90.1
- new net: DA2.1 (K), DA7.2 (A), R90.2
- new net: C40.1, P2.7 (Pin_7), R88.1
- new net: DA3.1 (K), DA8.2 (A), R82.2, R88.2
- new net: C41.1, P2.8 (Pin_8), R89.1
- new net: C39.1, P2.6 (Pin_6), R87.1
- new net: DA10.2 (A), DA5.1 (K), R78.2, R84.2
- new net: DA4.1 (K), DA9.2 (A), R80.2, R86.2
- new net: C43.1, P2.10 (Pin_10), R91.1
- new net: C35.1, P2.2 (Pin_2), R83.1
- new net: C36.1, P2.3 (Pin_3), R84.1
- new net: C37.1, P2.4 (Pin_4), R85.1
- new net: C38.1, P2.5 (Pin_5), R86.1
Other:
- moved on the sheet: C30, C31, C34, C81, C92, C93, C94, C95, C97, DB1, F1, J1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

Commit message: keep gerber folder
Connections:
- net at C34.1, U12.1 (IN): now also P3.1 (Pin_1); no longer P3.2 (Pin_2)
- net at C30.1, J1.2: now also T1.2; no longer T1.1
- net at C30.2, J1.1: now also T1.1; no longer T1.2
- net at C31.1, DB1.2: now also T1.4; no longer T1.3
- net at C31.2, DB1.3: now also T1.3; no longer T1.4
- net at F1.2: now also P3.2 (Pin_2); no longer P3.1 (Pin_1)
Other:
- moved on the sheet: P3, T1
Changed lines of the file:
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@@
     )
   )
-  (symbol (lib_id "Connector:Conn_01x02_Male") (at 425.45 34.29 270) (mirror x) (unit 1)
-    (in_bom yes) (on_board yes) (dnp no) (fields_autoplaced)
-    (property "Reference" "P3" (at 426.72 32.3849 90)
-      (effects (font (size 1.27 1.27)) (justify left))
-    )
-    (property "Value" "Conn_01x02_Male" (at 426.72 34.9249 90)
-      (effects (font (size 1.27 1.27)) (justify left))
-    )
-    (property "Footprint" "Connector_JST:JST_XH_B2B-XH-A_1x02_P2.50mm_Vertical" (at 425.45 34.29 0)
-      (effects (font (size 1.27 1.27)) hide)
-    )
-    (property "Datasheet" "~" (at 425.45 34.29 0)
+  (symbol (lib_id "Connector:Conn_01x02_Male") (at 422.91 34.29 90) (unit 1)
+    (in_bom yes) (on_board yes) (dnp no)
+    (property "Reference" "P3" (at 426.72 34.29 90)
+      (effects (font (size 1.27 1.27)) (justify right))
+    )
+    (property "Value" "Conn_01x02_Male" (at 426.72 31.75 90)
+      (effects (font (size 1.27 1.27)) (justify right))
+    )
+    (property "Footprint" "Connector_JST:JST_XH_B2B-XH-A_1x02_P2.50mm_Vertical" (at 422.91 34.29 0)
+      (effects (font (size 1.27 1.27)) hide)
+    )
+    (property "Datasheet" "~" (at 422.91 34.29 0)
       (effects (font (size 1.27 1.27)) hide)
     )
@@
     )
   )
-  (symbol (lib_id "Device:L_Coupled_1324") (at 501.65 31.75 0) (mirror y) (unit 1)
-    (in_bom yes) (on_board yes) (dnp no) (fields_autoplaced)
-    (property "Reference" "T1" (at 502.031 24.13 0)
-      (effects (font (size 1.27 1.27)))
-    )
-    (property "Value" "L_Coupled" (at 502.031 26.67 0)
-      (effects (font (size 1.27 1.27)))
-    )
+  (symbol (lib_id "Device:L_Coupled_1324") (at 501.65 31.75 180) (unit 1)
+    (in_bom yes) (on_board yes) (dnp no)
+    (property "Reference" "T1" (at 502.031 39.37 0)
+      (effects (font (size 1.27 1.27)))
+    )
+    (property "Value" "L_Coupled" (at 502.031 36.83 0)
+      (effects (font (size 1.27 1.27)))
+    )
