File: nonSNES.kicad_sch (KiCad schematic)
At the start: 62 parts, among them J1 Jack-DC, P1 CASSETTE, P2 Conn_2Rows-11Pins, P3 Conn_01x02_Male, SW1 RESET SW, T1 L_Coupled, U1 CPU, U12 L7805, U2 PPU1, U3 PPU2, U4 MS62256CL-10FC, U5 MS62256CL-10FC, U6 WRAM, U8 CIC, X1 Crystal

Commit message: dsp
Parts:
- added C63, C64: C_Polarized, Capacitor_SMD:CP_Elec_6.3x3, symbol Device:C_Polarized
- added U14: ~, Package_QFP:TQFP-64_14x14mm_P0.8mm, symbol SNES_Library:S-DSP
- added VA1: Varistor, Diode_SMD:D_3220_8050Metric, symbol Device:Varistor
- C67: value 1000u -> 2200u
Changed lines of the file:
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@@
   (symbol (lib_id "Device:C_Polarized") (at 342.265 38.735 0) (unit 1)
     (in_bom yes) (on_board yes) (dnp no) (fields_autoplaced)
-    (property "Reference" "C67" (at 345.44 37.211 0)
-      (effects (font (size 1.27 1.27)) (justify left))
-    )
-    (property "Value" "1000u" (at 345.44 39.751 0)
+    (property "Reference" "C67" (at 345.44 36.576 0)
+      (effects (font (size 1.27 1.27)) (justify left))
+    )
+    (property "Value" "2200u" (at 345.44 39.116 0)
       (effects (font (size 1.27 1.27)) (justify left))
     )
@@
         (path "/d1480d56-b791-43e1-bd4c-b0c74bb0533d"
           (reference "P1") (unit 1)
+        )
+      )
+    )
+  )
+  (symbol (lib_id "SNES_Library:S-DSP") (at 248.92 339.09 0) (unit 1)
+    (in_bom yes) (on_board yes) (dnp no) (fields_autoplaced)
+    (property "Reference" "U14" (at 248.285 308.61 0)
+      (effects (font (size 1.27 1.27)))
+    )
+    (property "Value" "~" (at 238.76 313.055 0)
+      (effects (font (size 1.27 1.27)))
+    )
+    (property "Footprint" "Package_QFP:TQFP-64_14x14mm_P0.8mm" (at 238.76 313.055 0)
+      (effects (font (size 1.27 1.27)) hide)
+    )
+    (property "Datasheet" "" (at 238.76 313.055 0)
+      (effects (font (size 1.27 1.27)) hide)
+    )
+    (pin "1")
+    (pin "10")
+    (pin "11")
+    (pin "12")
+    (pin "13")
+    (pin "14")
+    (pin "15")
+    (pin "16")
+    (pin "17")
+    (pin "18")
+    (pin "19")
+    (pin "2")
+    (pin "20")
+    (pin "21")
+    (pin "22")
+    (pin "23")
+    (pin "24")
+    (pin "25")
+    (pin "26")
+    (pin "27")
+    (pin "28")
+    (pin "29")
+    (pin "3")
+    (pin "30")
+    (pin "31")
+    (pin "32")
+    (pin "33")
+    (pin "34")
+    (pin "35")
+    (pin "36")
+    (pin "37")
+    (pin "38")
+    (pin "39")
+    (pin "4")
+    (pin "40")
+    (pin "41")
+    (pin "42")
+    (pin "43")
+    (pin "44")
+    (pin "45")
+    (pin "46")
+    (pin "47")
+    (pin "48")
+    (pin "49")
+    (pin "5")
+    (pin "50")
+    (pin "51")
+    (pin "52")
+    (pin "53")
+    (pin "54")
+    (pin "55")
+    (pin "56")
+    (pin "57")
+    (pin "58")
+    (pin "59")
+    (pin "6")
+    (pin "60")
+    (pin "61")
+    (pin "62")
+    (pin "63")
+    (pin "64")
+    (pin "7")
+    (pin "8")
+    (pin "9")
+    (instances
+      (project "nonSNES"
+        (path "/d1480d56-b791-43e1-bd4c-b0c74bb0533d"
+          (reference "U14") (unit 1)
         )
       )
@@
     )
   )
+  (symbol (lib_id "Device:C_Polarized") (at 353.06 74.93 0) (unit 1)
+    (in_bom yes) (on_board yes) (dnp no) (fields_autoplaced)
+    (property "Reference" "C64" (at 356.87 72.771 0)
+      (effects (font (size 1.27 1.27)) (justify left))
+    )
+    (property "Value" "C_Polarized" (at 356.87 75.311 0)
+      (effects (font (size 1.27 1.27)) (justify left))
+    )
+    (property "Footprint" "Capacitor_SMD:CP_Elec_6.3x3" (at 354.0252 78.74 0)
+      (effects (font (size 1.27 1.27)) hide)
+    )
+    (property "Datasheet" "~" (at 353.06 74.93 0)
+      (effects (font (size 1.27 1.27)) hide)
+    )
+    (pin "1")
+    (pin "2")
+    (instances
+      (project "nonSNES"
+        (path "/d1480d56-b791-43e1-bd4c-b0c74bb0533d"
+          (reference "C64") (unit 1)
+        )
+      )
+    )
+  )
   (symbol (lib_id "Device:C_Polarized") (at 66.04 72.39 0) (unit 1)
     (in_bom yes) (on_board yes) (dnp no)
@@
         (path "/d1480d56-b791-43e1-bd4c-b0c74bb0533d"
           (reference "P4") (unit 1)
+        )
+      )
+    )
+  )
+  (symbol (lib_id "Device:C_Polarized") (at 346.71 63.5 0) (unit 1)
+    (in_bom yes) (on_board yes) (dnp no) (fields_autoplaced)
+    (property "Reference" "C63" (at 350.52 61.341 0)
+      (effects (font (size 1.27 1.27)) (justify left))
+    )
+    (property "Value" "C_Polarized" (at 350.52 63.881 0)
+      (effects (font (size 1.27 1.27)) (justify left))
+    )
+    (property "Footprint" "Capacitor_SMD:CP_Elec_6.3x3" (at 347.6752 67.31 0)
+      (effects (font (size 1.27 1.27)) hide)
+    )
+    (property "Datasheet" "~" (at 346.71 63.5 0)
+      (effects (font (size 1.27 1.27)) hide)
+    )
+    (pin "1")
+    (pin "2")
+    (instances
+      (project "nonSNES"
+        (path "/d1480d56-b791-43e1-bd4c-b0c74bb0533d"
+          (reference "C63") (unit 1)
         )
       )
@@
         )
       )
+    )
+  )
+  (symbol (lib_id "Device:Varistor") (at 426.72 53.34 0) (unit 1)
+    (in_bom yes) (on_board yes) (dnp no) (fields_autoplaced)
+    (property "Reference" "VA1" (at 429.26 52.2633 0)
+      (effects (font (size 1.27 1.27)) (justify left))
+    )
+    (property "Value" "Varistor" (at 429.26 54.8033 0)
+      (effects (font (size 1.27 1.27)) (justify left))
+    )
+    (property "Footprint" "Diode_SMD:D_3220_8050Metric" (at 424.942 53.34 90)
+      (effects (font (size 1.27 1.27)) hide)
+    )
+    (property "Datasheet" "~" (at 426.72 53.34 0)
+      (effects (font (size 1.27 1.27)) hide)
+    )
+    (property "Sim.Name" "kicad_builtin_varistor" (at 426.72 53.34 0)
+      (effects (font (size 1.27 1.27)) hide)
+    )
+    (property "Sim.Device" "SUBCKT" (at 426.72 53.34 0)
+      (effects (font (size 1.27 1.27)) hide)
+    )
+    (property "Sim.Pins" "1=A 2=B" (at 426.72 53.34 0)
+      (effects (font (size 1.27 1.27)) hide)
+    )
+    (property "Sim.Params" "threshold=1k" (at 426.72 53.34 0)
+      (effects (font (size 1.27 1.27)) hide)
+    )
+    (property "Sim.Library" "${KICAD7_SYMBOL_DIR}/Simulation_SPICE.sp" (at 426.72 53.34 0)
+      (effects (font (size 1.27 1.27)) hide)
+    )
+    (pin "1")
+    (pin "2")
+    (instances
+      (project "nonSNES"
+        (path "/d1480d56-b791-43e1-bd4c-b0c74bb0533d"
+          (reference "VA1") (unit 1)
+        )
+      )

Commit message: s-enc
Parts:
- added U15, U16: MS62256CL-10FC, Package_SO:SOIC-28W_7.5x17.9mm_P1.27mm, symbol Memory_RAM:KM62256CLP
- added U7: ~, Package_SO:SO-24_5.3x15mm_P1.27mm, symbol SNES_Library:ENC
- renumbered U7 to J2

Commit message: sound
Parts:
- added U10: LM324, Package_SO:SO-14_3.9x8.65mm_P1.27mm, symbol Amplifier_Operational:LM324
- added U13: S-SMP, Package_QFP:LQFP-64_14x14mm_P0.8mm, symbol SNES_Library:S-SMP
- U14: footprint Package_QFP:TQFP-64_14x14mm_P0.8mm -> Package_QFP:PQFP-80_14x20mm_P0.8mm
Connections:
- net at U14.48 (CPUK): now also U13.16 (CPUK)
- net at U14.49 (PD2): now also U13.15 (PD2)
- net at U14.50 (PD3): now also U13.14 (PD3)
- net at U14.51 (D0): now also U13.13 (CPUD0)
- net at U14.53 (D1): now also U13.12 (CPUD1)
- net at U14.54 (D2): now also U13.11 (CPUD2)
- net at U14.55 (D3): now also U13.10 (CPUD3)
- net at U14.56 (D4): now also U13.9 (CPUD4)
- net at U14.57 (D5): now also U13.8 (CPUD5)
- net at U14.58 (D6): now also U13.7 (CPUD6)
- net at U14.59 (D7): now also U13.6 (CPUD7)
- net at U14.60 (A0): now also U13.5 (CPUA0)
- net at U14.61 (A1): now also U13.4 (CPUA1)
- net at U14.62 (A2): now also U13.3 (CPUA2)
- net at U14.63 (A3): now also U13.2 (CPUA3)
- net at U14.64 (A4): now also U13.1 (CPUA4)
- new net: U13.64 (CPUA5), U14.65 (A5)
- new net: U13.63 (CPUA6), U14.66 (A6)
- new net: U13.62 (CPUA7), U14.67 (A7)
- new net: U13.61 (CPUA8), U14.68 (A8)
- new net: U13.60 (CPUA9), U14.69 (A9)
- new net: U13.59 (CPUA10), U14.70 (A10)
- new net: U13.56 (CPUA11), U14.71 (A11)
- new net: U13.55 (CPUA12), U14.72 (A12)
- new net: U13.54 (CPUA13), U14.74 (A13)
- new net: U13.53 (CPUA14), U14.75 (A14)
- new net: U13.52 (CPUA15), U14.76 (A15)
