File: nonSNES.kicad_sch (KiCad schematic)
At the start: 310 parts, among them J1 Jack-DC, P1 CASSETTE, P2 Conn_2Rows-11Pins, P3 Conn_01x02_Pin, Q10 C2412K, Q11 C2412K, Q12 C2412K, Q13 Q_NPN_BEC, Q14 C2412K, Q15 C2412K, Q16 Q_NPN_BEC, Q17 Q_NPN_BEC, Q18 C2412, Q3 C2412K, Q4 C2412K, Q5 C2412K, Q6 C2412K, Q7 C2412K, Q8 C2412K, Q9 C2412K, SW1 RESET SW, T1 L_Coupled, U1 CPU, U10 LM324, U12 L7805, U13 S-SMP, U15 MS62256CL-10FC, U16 MS62256CL-10FC, U17 uPD6367, U2 PPU1, U3 PPU2, U4 MS62256CL-10FC, U5 MS62256CL-10FC, U6 WRAM, U8 CIC, X1 Crystal, X2 Crystal

Commit message: manufacturing data
Parts:
- C1, C3, C44, C45, C47, C48, C49, C50, C51, C52: value 47p -> 47pF
- C10, C11, C70: value 82p -> 82pF
- C100, C101, C29, C33, C34, C6, C69, C7, C8, C80, C82, C84, C88, C89, C90, C91, C98, C99: value 100n -> 100nF
- C13, C15: value 220p -> 220pF
- C14, C16, C18, C23, C24, C25, C26, C27, C28, C53, C54: value 1u -> 1uF
- C17, C19, C20, C86: value 10p -> 10pF
- C2, C4, C96: value 47p -> 47pF; now left out of the parts list
- C22, C35, C36, C37, C38, C39, C40, C41, C42, C43: value 330p -> 330pF
- C32: value 100 -> 100nF
- C46: value 330 -> 330pF
- C5: value 15p -> 15pF
- C59, C60, C61, C66: value 10u 50V -> 10uF 50V
- C62: value 2.2u -> 2.2uF
- C67: value 2200u -> 2200uF
- C68: value 56p -> 56pF
- C74, C77, C9: value 1n -> 1nF
- C75: value 1,8n -> 1800pF
- C76, C79: value 100p -> 100pF
- C78: value 1800p -> 1800pF
- C83: value 0.01u -> 0.01uF
- C85: value 0.1u -> 0.1uF
- C92, C93, C94: value C -> 0.1uF
- Q13, Q16, Q17: value Q_NPN_BEC -> C2412K
- Q18: value C2412 -> C2412K
- R106, R107, R2: value 5,1k -> 5.1k
- R108, R109, R110, R111, R24, R32, R4, R42, R45, R47, R5, R6, TP1, TP10, TP11, TP12, TP13, TP14, TP15, TP16, TP17, TP18, TP19, TP2, TP20, TP21, TP22, TP23, TP24, TP25, TP26, TP27, TP28, TP29, TP3, TP30, TP31, TP32, TP33, TP34, TP35, TP36, TP37, TP38, TP4, TP5, TP6, TP7, TP8, TP9: now left out of the parts list
- R13, R18, R8: value 1,1k -> 1.1k
- R14, R19, R9: value 1,5k -> 1.5k
- R26, R57, R64, R76: value 1,8k -> 1.8k
- R28, R29: value 3,3k -> 3.3k
- R74: value 2,2k -> 2.2k
Connections:
- net /IRQ: no longer P5.26 (~{IRQ}), TP21.1
- new net: P5.26 (~{IRQ}), TP21.1

Commit message: values
Parts:
- C63: value C_Polarized -> 33uF 25V
- C64: value 33u 25V -> 33uF 25V
- U17: value uPD6367 -> uPD6376
- X1: value Crystal -> 17.734MHz
- X2: value Crystal -> 24.576MHz
Changed lines of the file:
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@@
       (effects (font (size 1.27 1.27)) hide)
     )
-    (property "Datasheet" "~" (at 131.445 360.045 0)
+    (property "Datasheet" "GKG20067-07" (at 131.445 360.045 0)
       (effects (font (size 1.27 1.27)) hide)
     )
@@
       (effects (font (size 1.27 1.27)) (justify right))
     )
-    (property "Value" "Crystal" (at 139.7 377.825 90)
+    (property "Value" "17.734MHz" (at 139.7 377.825 90)
       (effects (font (size 1.27 1.27)) (justify right))
     )
@@
       (effects (font (size 1.27 1.27)))
     )
-    (property "Value" "uPD6367" (at 321.945 265.43 0)
+    (property "Value" "uPD6376" (at 321.945 265.43 0)
       (effects (font (size 1.27 1.27)))
     )
@@
       (effects (font (size 1.27 1.27)))
     )
-    (property "Value" "33u 25V" (at 399.034 15.24 90)
+    (property "Value" "33uF 25V" (at 399.034 15.24 90)
       (effects (font (size 1.27 1.27)))
     )
@@
   (symbol (lib_id "Device:Crystal") (at 308.61 302.895 0) (unit 1)
     (in_bom yes) (on_board yes) (dnp no) (fields_autoplaced)
-    (property "Reference" "X2" (at 308.61 295.275 0)
+    (property "Reference" "X2" (at 308.61 295.91 0)
       (effects (font (size 1.27 1.27)))
     )
-    (property "Value" "Crystal" (at 308.61 297.815 0)
+    (property "Value" "24.576MHz" (at 308.61 298.45 0)
       (effects (font (size 1.27 1.27)))
     )
@@
       (effects (font (size 1.27 1.27)) (justify left))
     )
-    (property "Value" "C_Polarized" (at 425.45 33.401 0)
+    (property "Value" "33uF 25V" (at 425.45 33.401 0)
       (effects (font (size 1.27 1.27)) (justify left))
     )

Commit message: references
Parts:
- added C102: 100nF, Capacitor_SMD:C_0805_2012Metric, symbol Device:C
- U14: value ~ -> S-DSP; footprint Package_QFP:PQFP-80_14x20mm_P0.8mm -> SNES_Library:PQFP-80_15x22mm_P0.8mm
- U18: value ~ -> S-CLK
Connections:
- net GND: now also C102.2
- net VCC: now also C102.1
Changed lines of the file:
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@@
     )
   )
+  (symbol (lib_id "power:VCC") (at 273.685 39.37 0) (unit 1)
+    (in_bom yes) (on_board yes) (dnp no) (fields_autoplaced)
+    (property "Reference" "#PWR0192" (at 273.685 43.18 0)
+      (effects (font (size 1.27 1.27)) hide)
+    )
+    (property "Value" "VCC" (at 273.685 34.29 0)
+      (effects (font (size 1.27 1.27)))
+    )
+    (property "Footprint" "" (at 273.685 39.37 0)
+      (effects (font (size 1.27 1.27)) hide)
+    )
+    (property "Datasheet" "" (at 273.685 39.37 0)
+      (effects (font (size 1.27 1.27)) hide)
+    )
+    (pin "1")
+    (instances
+      (project "nonSNES"
+        (path "/d1480d56-b791-43e1-bd4c-b0c74bb0533d"
+          (reference "#PWR0192") (unit 1)
+        )
+      )
+    )
+  )
   (symbol (lib_id "power:VCC") (at 337.82 198.12 0) (unit 1)
     (in_bom yes) (on_board yes) (dnp no) (fields_autoplaced)
@@
       (effects (font (size 1.27 1.27)))
     )
-    (property "Value" "~" (at 311.785 278.13 0)
+    (property "Value" "S-DSP" (at 311.785 278.13 0)
       (effects (font (size 1.27 1.27)))
     )
-    (property "Footprint" "Package_QFP:PQFP-80_14x20mm_P0.8mm" (at 311.785 278.13 0)
+    (property "Footprint" "SNES_Library:PQFP-80_15x22mm_P0.8mm" (at 311.785 278.13 0)
       (effects (font (size 1.27 1.27)) hide)
     )
@@
       (effects (font (size 1.27 1.27)))
     )
-    (property "Value" "~" (at 142.875 380.365 0)
+    (property "Value" "S-CLK" (at 142.875 380.365 0)
       (effects (font (size 1.27 1.27)))
     )
@@
     )
   )
+  (symbol (lib_id "Device:C") (at 277.495 39.37 90) (unit 1)
+    (in_bom yes) (on_board yes) (dnp no)
+    (property "Reference" "C102" (at 277.495 31.75 90)
+      (effects (font (size 1.27 1.27)))
+    )
+    (property "Value" "100nF" (at 277.495 34.29 90)
+      (effects (font (size 1.27 1.27)))
+    )
+    (property "Footprint" "Capacitor_SMD:C_0805_2012Metric" (at 281.305 38.4048 0)
+      (effects (font (size 1.27 1.27)) hide)
+    )
+    (property "Datasheet" "~" (at 277.495 39.37 0)
+      (effects (font (size 1.27 1.27)) hide)
+    )
+    (pin "1")
+    (pin "2")
+    (instances
+      (project "nonSNES"
+        (path "/d1480d56-b791-43e1-bd4c-b0c74bb0533d"
+          (reference "C102") (unit 1)
+        )
+      )
+    )
+  )
   (symbol (lib_id "Device:R") (at 344.805 209.55 0) (unit 1)
     (in_bom yes) (on_board yes) (dnp no)
@@
         )
       )
+    )
+  )
+  (symbol (lib_id "power:GND") (at 281.305 39.37 90) (unit 1)
+    (in_bom yes) (on_board yes) (dnp no) (fields_autoplaced)
+    (property "Reference" "#PWR0193" (at 287.655 39.37 0)
+      (effects (font (size 1.27 1.27)) hide)
+    )
+    (property "Value" "GND" (at 285.115 39.37 90)
+      (effects (font (size 1.27 1.27)) (justify right))
+    )
+    (property "Footprint" "" (at 281.305 39.37 0)
+      (effects (font (size 1.27 1.27)) hide)
+    )
+    (property "Datasheet" "" (at 281.305 39.37 0)
+      (effects (font (size 1.27 1.27)) hide)
+    )
+    (pin "1")
+    (instances
+      (project "nonSNES"
+        (path "/d1480d56-b791-43e1-bd4c-b0c74bb0533d"
+          (reference "#PWR0193") (unit 1)
+        )
+      )

Commit message: fix 100nF
Parts:
- C100, C101, C102, C29, C32, C33, C34, C6, C69, C7, C8, C80, C82, C84, C88, C89, C90, C91, C98, C99: value 100nF -> 0.1µF
- C31, C85, C92, C93, C94, C95, C97: value 0.1uF -> 0.1µF
- U7: value ~ -> S-ENC
Changed lines of the file:
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@@
       (effects (font (size 1.27 1.27)) (justify right))
     )
-    (property "Value" "100nF" (at 370.84 361.315 0)
+    (property "Value" "0.1µF" (at 370.84 361.315 0)
       (effects (font (size 1.27 1.27)) (justify right))
     )
@@
       (effects (font (size 1.27 1.27)) (justify left))
     )
-    (property "Value" "0.1uF" (at 270.51 121.92 0)
+    (property "Value" "0.1µF" (at 270.51 121.92 0)
       (effects (font (size 1.27 1.27)) (justify left))
     )
@@
       (effects (font (size 1.27 1.27)) (justify left))
     )
-    (property "Value" "100nF" (at 44.45 389.001 0)
+    (property "Value" "0.1µF" (at 44.45 389.001 0)
       (effects (font (size 1.27 1.27)) (justify left))
     )
@@
       (effects (font (size 1.27 1.27)))
     )
-    (property "Value" "0.1uF" (at 181.61 118.11 90)
+    (property "Value" "0.1µF" (at 181.61 118.11 90)
       (effects (font (size 1.27 1.27)))
     )
@@
     )
   )
-  (symbol (lib_id "power:VCC") (at 273.685 39.37 0) (unit 1)
-    (in_bom yes) (on_board yes) (dnp no) (fields_autoplaced)
-    (property "Reference" "#PWR0192" (at 273.685 43.18 0)
+  (symbol (lib_id "power:VCC") (at 273.685 39.37 90) (unit 1)
+    (in_bom yes) (on_board yes) (dnp no)
+    (property "Reference" "#PWR0192" (at 277.495 39.37 0)
       (effects (font (size 1.27 1.27)) hide)
     )
-    (property "Value" "VCC" (at 273.685 34.29 0)
-      (effects (font (size 1.27 1.27)))
+    (property "Value" "VCC" (at 267.335 39.37 90)
+      (effects (font (size 1.27 1.27)) (justify right))
     )
     (property "Footprint" "" (at 273.685 39.37 0)
@@
       (effects (font (size 1.27 1.27)) (justify right))
     )
-    (property "Value" "100nF" (at 440.69 177.165 0)
+    (property "Value" "0.1µF" (at 440.69 177.165 0)
       (effects (font (size 1.27 1.27)) (justify right))
     )
@@
       (effects (font (size 1.27 1.27)) (justify left))
     )
-    (property "Value" "100nF" (at 448.31 98.425 0)
+    (property "Value" "0.1µF" (at 448.31 98.425 0)
       (effects (font (size 1.27 1.27)) (justify left))
     )
@@
       (effects (font (size 1.27 1.27)) (justify left))
     )
-    (property "Value" "0.1uF" (at 487.68 34.2899 0)
+    (property "Value" "0.1µF" (at 487.68 34.2899 0)
       (effects (font (size 1.27 1.27)) (justify left))
     )
@@
       (effects (font (size 1.27 1.27)) (justify right))
     )
-    (property "Value" "100nF" (at 354.33 36.83 0)
+    (property "Value" "0.1µF" (at 354.33 36.83 0)
       (effects (font (size 1.27 1.27)) (justify right))
     )
@@
       (effects (font (size 1.27 1.27)) (justify left))
     )
-    (property "Value" "100nF" (at 400.05 36.83 0)
+    (property "Value" "0.1µF" (at 400.05 36.83 0)
       (effects (font (size 1.27 1.27)) (justify left))
     )
@@
       (effects (font (size 1.27 1.27)))
     )
-    (property "Value" "100nF" (at 302.895 180.975 90)
+    (property "Value" "0.1µF" (at 302.895 180.975 90)
       (effects (font (size 1.27 1.27)))
     )
@@
       (effects (font (size 1.27 1.27)) (justify right))
     )
-    (property "Value" "100nF" (at 177.8 375.92 0)
+    (property "Value" "0.1µF" (at 177.8 375.92 0)
       (effects (font (size 1.27 1.27)) (justify right))
     )
@@
       (effects (font (size 1.27 1.27)) (justify right))
     )
-    (property "Value" "100nF" (at 370.84 323.85 0)
+    (property "Value" "0.1µF" (at 370.84 323.85 0)
       (effects (font (size 1.27 1.27)) (justify right))
     )
@@
       (effects (font (size 1.27 1.27)) (justify right))
     )
-    (property "Value" "100nF" (at 381 234.315 0)
+    (property "Value" "0.1µF" (at 381 234.315 0)
       (effects (font (size 1.27 1.27)) (justify right))
     )
@@
       (effects (font (size 1.27 1.27)))
     )
-    (property "Value" "~" (at 420.37 134.62 0)
+    (property "Value" "S-ENC" (at 420.37 134.62 0)
       (effects (font (size 1.27 1.27)))
     )
@@
       (effects (font (size 1.27 1.27)) hide)
     )
-    (property "Datasheet" "" (at 420.37 134.62 0)
+    (property "Datasheet" "https://wiki.console5.com/tw/images/e/e6/BA6592F.pdf" (at 420.37 134.62 0)
       (effects (font (size 1.27 1.27)) hide)
     )
@@
       (effects (font (size 1.27 1.27)))
     )
-    (property "Value" "100nF" (at 316.23 151.765 90)
+    (property "Value" "0.1µF" (at 316.23 151.765 90)
       (effects (font (size 1.27 1.27)))
     )
@@
       (effects (font (size 1.27 1.27)) (justify left))
     )
-    (property "Value" "0.1uF" (at 81.28 371.221 0)
+    (property "Value" "0.1µF" (at 81.28 371.221 0)
       (effects (font (size 1.27 1.27)) (justify left))
     )
@@
       (effects (font (size 1.27 1.27)) (justify right))
     )
-    (property "Value" "100nF" (at 21.59 274.32 0)
+    (property "Value" "0.1µF" (at 21.59 274.32 0)
       (effects (font (size 1.27 1.27)) (justify right))
     )
@@
       (effects (font (size 1.27 1.27)))
     )
-    (property "Value" "100nF" (at 325.755 277.495 90)
+    (property "Value" "0.1µF" (at 325.755 277.495 90)
       (effects (font (size 1.27 1.27)))
     )
@@
       (effects (font (size 1.27 1.27)))
     )
-    (property "Value" "100nF" (at 318.135 277.495 90)
+    (property "Value" "0.1µF" (at 318.135 277.495 90)
       (effects (font (size 1.27 1.27)))
     )
@@
       (effects (font (size 1.27 1.27)) (justify left))
     )
-    (property "Value" "0.1uF" (at 82.55 121.285 0)
+    (property "Value" "0.1µF" (at 82.55 121.285 0)
       (effects (font (size 1.27 1.27)) (justify left))
     )
@@
       (effects (font (size 1.27 1.27)))
     )
-    (property "Value" "100nF" (at 277.495 34.29 90)
+    (property "Value" "0.1µF" (at 277.495 34.29 90)
       (effects (font (size 1.27 1.27)))
     )
@@
       (effects (font (size 1.27 1.27)) (justify left))
     )
-    (property "Value" "100nF" (at 389.89 36.83 0)
+    (property "Value" "0.1µF" (at 389.89 36.83 0)
       (effects (font (size 1.27 1.27)) (justify left))
     )
@@
       (effects (font (size 1.27 1.27)))
     )
-    (property "Value" "100nF" (at 265.43 305.435 90)
+    (property "Value" "0.1µF" (at 265.43 305.435 90)
       (effects (font (size 1.27 1.27)))
     )
@@
       (effects (font (size 1.27 1.27)) (justify left))
     )
-    (property "Value" "0.1uF" (at 142.24 121.92 0)
+    (property "Value" "0.1µF" (at 142.24 121.92 0)
       (effects (font (size 1.27 1.27)) (justify left))
     )
@@
       (effects (font (size 1.27 1.27)))
     )
-    (property "Value" "0.1uF" (at 181.61 175.26 90)
+    (property "Value" "0.1µF" (at 181.61 175.26 90)
       (effects (font (size 1.27 1.27)))
     )
@@
       (effects (font (size 1.27 1.27)) (justify left))
     )
-    (property "Value" "100nF" (at 446.405 41.91 0)
+    (property "Value" "0.1µF" (at 446.405 41.91 0)
       (effects (font (size 1.27 1.27)) (justify left))
     )
@@
       (effects (font (size 1.27 1.27)))
     )
-    (property "Value" "100nF" (at 207.645 53.34 90)
+    (property "Value" "0.1µF" (at 207.645 53.34 90)
       (effects (font (size 1.27 1.27)))
     )
@@
       (effects (font (size 1.27 1.27)))
     )
-    (property "Value" "100nF" (at 350.52 208.915 90)
+    (property "Value" "0.1µF" (at 350.52 208.915 90)
       (effects (font (size 1.27 1.27)))
     )

Commit message: fix errors
Parts:
- renumbered C20 to C12
Connections:
- net /IRQ: now also P5.26 (~{IRQ}), TP21.1
Changed lines of the file:
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@@
     )
   )
-  (global_label "{slash}IRQ" (shape input) (at 159.385 311.15 0) (fields_autoplaced)
+  (global_label "{slash}IRQ" (shape input) (at 158.75 311.15 0) (fields_autoplaced)
     (effects (font (size 1.27 1.27)) (justify left))
-    (property "Intersheetrefs" "${INTERSHEET_REFS}" (at 166.906 311.15 0)
+    (property "Intersheetrefs" "${INTERSHEET_REFS}" (at 166.271 311.15 0)
       (effects (font (size 1.27 1.27)) (justify left) hide)
     )
@@
   (symbol (lib_id "Device:C") (at 516.255 149.225 0) (unit 1)
     (in_bom yes) (on_board yes) (dnp no)
-    (property "Reference" "C20" (at 518.795 147.955 0)
+    (property "Reference" "C12" (at 518.795 147.955 0)
       (effects (font (size 1.27 1.27)) (justify left))
     )
@@
       (project "nonSNES"
         (path "/d1480d56-b791-43e1-bd4c-b0c74bb0533d"
-          (reference "C20") (unit 1)
+          (reference "C12") (unit 1)
         )
       )

Commit message: flip around most of the silkscreen on the bottom
Parts:
- renumbered C5 to C2, C2 to C5, C96 to C69, C69 to C96
Changed lines of the file:
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@@
   (symbol (lib_id "Device:C") (at 170.815 402.59 0) (mirror y) (unit 1)
     (in_bom no) (on_board yes) (dnp yes)
-    (property "Reference" "C96" (at 163.83 402.59 90)
+    (property "Reference" "C69" (at 163.83 402.59 90)
       (effects (font (size 1.27 1.27)))
     )
@@
       (project "nonSNES"
         (path "/d1480d56-b791-43e1-bd4c-b0c74bb0533d"
-          (reference "C96") (unit 1)
+          (reference "C69") (unit 1)
         )
       )
@@
   (symbol (lib_id "Device:C") (at 351.155 35.56 180) (unit 1)
     (in_bom yes) (on_board yes) (dnp no) (fields_autoplaced)
-    (property "Reference" "C69" (at 354.33 34.29 0)
+    (property "Reference" "C96" (at 354.33 34.29 0)
       (effects (font (size 1.27 1.27)) (justify right))
     )
@@
       (project "nonSNES"
         (path "/d1480d56-b791-43e1-bd4c-b0c74bb0533d"
-          (reference "C69") (unit 1)
+          (reference "C96") (unit 1)
         )
       )
@@
   (symbol (lib_id "Device:C") (at 131.445 387.985 90) (mirror x) (unit 1)
     (in_bom no) (on_board yes) (dnp yes)
-    (property "Reference" "C2" (at 131.445 394.97 90)
+    (property "Reference" "C5" (at 131.445 394.97 90)
       (effects (font (size 1.27 1.27)))
     )
@@
       (project "nonSNES"
         (path "/d1480d56-b791-43e1-bd4c-b0c74bb0533d"
-          (reference "C2") (unit 1)
+          (reference "C5") (unit 1)
         )
       )
@@
   (symbol (lib_id "Device:C") (at 131.445 370.84 90) (unit 1)
     (in_bom yes) (on_board yes) (dnp no) (fields_autoplaced)
-    (property "Reference" "C5" (at 131.445 363.22 90)
+    (property "Reference" "C2" (at 131.445 363.22 90)
       (effects (font (size 1.27 1.27)))
     )
@@
       (project "nonSNES"
         (path "/d1480d56-b791-43e1-bd4c-b0c74bb0533d"
-          (reference "C5") (unit 1)
+          (reference "C2") (unit 1)
         )
       )
