File: nonSNES.kicad_pcb (KiCad board)
At the start: 4 copper layers, 185.4 x 160 mm, 13 parts, among them J1 Jack-DC, P3 Conn_01x02_Male, T1 L_Coupled, U1 CPU, U12 L7805, U2 PQFP-100_14x20mm_P0.65mm, U3 PQFP-100_14x20mm_P0.65mm, U4 SOIC-28W_7.5x17.9mm_P1.27mm, U5 SOIC-28W_7.5x17.9mm_P1.27mm

Commit message: replace footprints
Parts:
- added C34: 0.1uF, Capacitor_SMD:C_0805_2012Metric, F.Cu at (71.1, 160.0)
- added C81: 1uF, Capacitor_SMD:C_0805_2012Metric, F.Cu at (75.6, 160.0)
- J1: footprint Connector_Molex:Molex_Mega-Fit_76829-0102_2x01_P5.70mm_Vertical -> SNES_Library:DcJack
- U4, U5: value SOIC-28W_7.5x17.9mm_P1.27mm -> KM62256CLP
- moved J1 7.74 mm to (30.5, 167.6), turned to 0 degrees
- moved T1 2.54 mm to (35.6, 157.5)
Connections:
- U12 pad 2: unconnected-(U12-Pad2) -> GNDPWR
- U12 pad 3: unconnected-(U12-Pad3) -> VCC
- U4 pad 1: (no net) -> unconnected-(U4-Pad1)
- U4 pad 10: (no net) -> unconnected-(U4-Pad10)
- U4 pad 11: (no net) -> unconnected-(U4-Pad11)
- U4 pad 12: (no net) -> unconnected-(U4-Pad12)
- U4 pad 13: (no net) -> unconnected-(U4-Pad13)
- U4 pad 14: (no net) -> unconnected-(U4-Pad14)
- U4 pad 15: (no net) -> unconnected-(U4-Pad15)
- U4 pad 16: (no net) -> unconnected-(U4-Pad16)
- U4 pad 17: (no net) -> unconnected-(U4-Pad17)
- U4 pad 18: (no net) -> unconnected-(U4-Pad18)
- U4 pad 19: (no net) -> unconnected-(U4-Pad19)
- U4 pad 2: (no net) -> unconnected-(U4-Pad2)
- U4 pad 20: (no net) -> unconnected-(U4-Pad20)
- U4 pad 21: (no net) -> unconnected-(U4-Pad21)
- U4 pad 22: (no net) -> unconnected-(U4-Pad22)
- U4 pad 23: (no net) -> unconnected-(U4-Pad23)
- U4 pad 24: (no net) -> unconnected-(U4-Pad24)
- U4 pad 25: (no net) -> unconnected-(U4-Pad25)
- U4 pad 26: (no net) -> unconnected-(U4-Pad26)
- U4 pad 27: (no net) -> unconnected-(U4-Pad27)
- U4 pad 28: (no net) -> unconnected-(U4-Pad28)
- U4 pad 3: (no net) -> unconnected-(U4-Pad3)
- U4 pad 4: (no net) -> unconnected-(U4-Pad4)
- U4 pad 5: (no net) -> unconnected-(U4-Pad5)
- U4 pad 6: (no net) -> unconnected-(U4-Pad6)
- U4 pad 7: (no net) -> unconnected-(U4-Pad7)
- U4 pad 8: (no net) -> unconnected-(U4-Pad8)
- U4 pad 9: (no net) -> unconnected-(U4-Pad9)
- U5 pad 1: (no net) -> unconnected-(U5-Pad1)
- U5 pad 10: (no net) -> unconnected-(U5-Pad10)
- U5 pad 11: (no net) -> unconnected-(U5-Pad11)
- U5 pad 12: (no net) -> unconnected-(U5-Pad12)
- U5 pad 13: (no net) -> unconnected-(U5-Pad13)
- U5 pad 14: (no net) -> unconnected-(U5-Pad14)
- U5 pad 15: (no net) -> unconnected-(U5-Pad15)
- U5 pad 16: (no net) -> unconnected-(U5-Pad16)
- U5 pad 17: (no net) -> unconnected-(U5-Pad17)
- U5 pad 18: (no net) -> unconnected-(U5-Pad18)
- U5 pad 19: (no net) -> unconnected-(U5-Pad19)
- U5 pad 2: (no net) -> unconnected-(U5-Pad2)
- U5 pad 20: (no net) -> unconnected-(U5-Pad20)
- U5 pad 21: (no net) -> unconnected-(U5-Pad21)
- U5 pad 22: (no net) -> unconnected-(U5-Pad22)
- U5 pad 23: (no net) -> unconnected-(U5-Pad23)
- U5 pad 24: (no net) -> unconnected-(U5-Pad24)
- U5 pad 25: (no net) -> unconnected-(U5-Pad25)
- U5 pad 26: (no net) -> unconnected-(U5-Pad26)
- U5 pad 27: (no net) -> unconnected-(U5-Pad27)
- U5 pad 28: (no net) -> unconnected-(U5-Pad28)
- U5 pad 3: (no net) -> unconnected-(U5-Pad3)
- U5 pad 4: (no net) -> unconnected-(U5-Pad4)
- U5 pad 5: (no net) -> unconnected-(U5-Pad5)
- U5 pad 6: (no net) -> unconnected-(U5-Pad6)
- U5 pad 7: (no net) -> unconnected-(U5-Pad7)
- U5 pad 8: (no net) -> unconnected-(U5-Pad8)
- U5 pad 9: (no net) -> unconnected-(U5-Pad9)
Other:
- outline, holes or cut-outs redrawn

Commit message: connect vram data lines
Parts:
- added C93: C, Capacitor_SMD:C_0805_2012Metric, B.Cu at (165.1, 147.3)
- added C95: 0.1uF, Capacitor_SMD:C_0805_2012Metric, B.Cu at (144.8, 68.6)
- added C97: 0.1uF, Capacitor_SMD:C_0805_2012Metric, B.Cu at (172.7, 67.6)
- added P1: CASSETTE, Connector_DIN:DIN41612_R_2x32_Male_Vertical_THT, F.Cu at (95.3, 137.2)
- U4, U5: value KM62256CLP -> MS62256CL-10FC
- moved U2 27.0 mm to (172.7, 94.0)
- moved U3 25.1 mm to (142.2, 94.0)
- moved U4 25.1 mm to (172.7, 68.6)
- moved U5 25.1 mm to (144.8, 68.6)
- moved U1 16.1 mm to (165.1, 147.3)
Connections:
- U1 pad 1: unconnected-(U1-Pad1) -> VCC
- U1 pad 34: unconnected-(U1-Pad34) -> VCC
- U4 pad 11: unconnected-(U4-Pad11) -> /D0
- U4 pad 12: unconnected-(U4-Pad12) -> /D1
- U4 pad 13: unconnected-(U4-Pad13) -> /D2
- U4 pad 14: unconnected-(U4-Pad14) -> GNDPWR
- U4 pad 15: unconnected-(U4-Pad15) -> /D3
- U4 pad 16: unconnected-(U4-Pad16) -> /D4
- U4 pad 17: unconnected-(U4-Pad17) -> /D5
- U4 pad 18: unconnected-(U4-Pad18) -> /D6
- U4 pad 19: unconnected-(U4-Pad19) -> /D7
- U4 pad 20: unconnected-(U4-Pad20) -> GNDPWR
- U4 pad 28: unconnected-(U4-Pad28) -> VCC
- U5 pad 11: unconnected-(U5-Pad11) -> /D0
- U5 pad 12: unconnected-(U5-Pad12) -> /D1
- U5 pad 13: unconnected-(U5-Pad13) -> /D2
- U5 pad 14: unconnected-(U5-Pad14) -> GNDPWR
- U5 pad 15: unconnected-(U5-Pad15) -> /D3
- U5 pad 16: unconnected-(U5-Pad16) -> /D4
- U5 pad 17: unconnected-(U5-Pad17) -> /D5
- U5 pad 18: unconnected-(U5-Pad18) -> /D6
- U5 pad 19: unconnected-(U5-Pad19) -> /D7
- U5 pad 20: unconnected-(U5-Pad20) -> GNDPWR
- U5 pad 28: unconnected-(U5-Pad28) -> VCC

Commit message: get board outline right
Parts:
- moved C93 55.3 mm to (212.1, 176.5)
- moved C95 55.3 mm to (191.8, 97.8)
- moved C97 55.3 mm to (219.7, 96.8)
- moved P1 55.3 mm to (142.3, 166.4)
- moved U1 55.3 mm to (212.1, 176.5)
- moved U4 55.3 mm to (219.7, 97.8)
- moved U5 55.3 mm to (191.8, 97.8)
- moved C30 55.3 mm to (85.1, 196.8)
- moved P3 55.3 mm to (102.9, 196.4)
- moved U2 55.3 mm to (219.7, 123.2)
- moved C81 55.3 mm to (122.6, 189.2)
- moved DB1 55.3 mm to (105.4, 174.0)
- moved J1 55.3 mm to (77.5, 196.8)
- moved T1 55.3 mm to (82.5, 186.7)
- moved U12 55.3 mm to (115.6, 196.8)
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Other:
- board size 185.4 x 160 mm -> 188 x 161.3 mm

Commit message: place ppu
Parts:
- added C92: C, Capacitor_SMD:C_0805_2012Metric, B.Cu at (188.6, 122.6)
- added C94: C, Capacitor_SMD:C_0805_2012Metric, B.Cu at (219.1, 118.7)
- U2: value PQFP-100_14x20mm_P0.65mm -> PPU1
- U3: value PQFP-100_14x20mm_P0.65mm -> PPU2
- moved U1 7.73 mm to (213.4, 168.9)
- moved C93 6.42 mm to (213.0, 170.2)
Connections:
- U1 pad 59: unconnected-(U1-Pad59) -> VCC
- U1 pad 85: unconnected-(U1-Pad85) -> VCC
- U2 pad 1: (no net) -> unconnected-(U2-Pad1)
- U2 pad 10: (no net) -> unconnected-(U2-Pad10)
- U2 pad 100: (no net) -> unconnected-(U2-Pad100)
- U2 pad 11: (no net) -> unconnected-(U2-Pad11)
- U2 pad 12: (no net) -> unconnected-(U2-Pad12)
- U2 pad 13: (no net) -> VCC
- U2 pad 14: (no net) -> unconnected-(U2-Pad14)
- U2 pad 15: (no net) -> unconnected-(U2-Pad15)
- U2 pad 16: (no net) -> unconnected-(U2-Pad16)
- U2 pad 17: (no net) -> unconnected-(U2-Pad17)
- U2 pad 18: (no net) -> unconnected-(U2-Pad18)
- U2 pad 19: (no net) -> unconnected-(U2-Pad19)
- U2 pad 2: (no net) -> unconnected-(U2-Pad2)
- U2 pad 20: (no net) -> unconnected-(U2-Pad20)
- U2 pad 21: (no net) -> unconnected-(U2-Pad21)
- U2 pad 22: (no net) -> unconnected-(U2-Pad22)
- U2 pad 23: (no net) -> unconnected-(U2-Pad23)
- U2 pad 24: (no net) -> unconnected-(U2-Pad24)
- U2 pad 25: (no net) -> unconnected-(U2-Pad25)
- U2 pad 26: (no net) -> unconnected-(U2-Pad26)
- U2 pad 27: (no net) -> unconnected-(U2-Pad27)
- U2 pad 28: (no net) -> unconnected-(U2-Pad28)
- U2 pad 29: (no net) -> unconnected-(U2-Pad29)
- U2 pad 3: (no net) -> unconnected-(U2-Pad3)
- U2 pad 30: (no net) -> unconnected-(U2-Pad30)
- U2 pad 31: (no net) -> unconnected-(U2-Pad31)
- U2 pad 32: (no net) -> unconnected-(U2-Pad32)
- U2 pad 33: (no net) -> unconnected-(U2-Pad33)
- U2 pad 34: (no net) -> unconnected-(U2-Pad34)
- U2 pad 35: (no net) -> unconnected-(U2-Pad35)
- U2 pad 36: (no net) -> VCC
- U2 pad 37: (no net) -> unconnected-(U2-Pad37)
- U2 pad 38: (no net) -> unconnected-(U2-Pad38)
- U2 pad 39: (no net) -> unconnected-(U2-Pad39)
- U2 pad 4: (no net) -> unconnected-(U2-Pad4)
- U2 pad 40: (no net) -> unconnected-(U2-Pad40)
- U2 pad 41: (no net) -> unconnected-(U2-Pad41)
- U2 pad 42: (no net) -> unconnected-(U2-Pad42)
- U2 pad 43: (no net) -> unconnected-(U2-Pad43)
- U2 pad 44: (no net) -> unconnected-(U2-Pad44)
- U2 pad 45: (no net) -> unconnected-(U2-Pad45)
- U2 pad 46: (no net) -> unconnected-(U2-Pad46)
- U2 pad 47: (no net) -> unconnected-(U2-Pad47)
- U2 pad 48: (no net) -> unconnected-(U2-Pad48)
- U2 pad 49: (no net) -> unconnected-(U2-Pad49)
- U2 pad 5: (no net) -> unconnected-(U2-Pad5)
- U2 pad 50: (no net) -> unconnected-(U2-Pad50)
- U2 pad 51: (no net) -> unconnected-(U2-Pad51)
- U2 pad 52: (no net) -> unconnected-(U2-Pad52)
- U2 pad 53: (no net) -> unconnected-(U2-Pad53)
- U2 pad 54: (no net) -> unconnected-(U2-Pad54)
- U2 pad 55: (no net) -> unconnected-(U2-Pad55)
- U2 pad 56: (no net) -> unconnected-(U2-Pad56)
- U2 pad 57: (no net) -> unconnected-(U2-Pad57)
- U2 pad 58: (no net) -> unconnected-(U2-Pad58)
- U2 pad 59: (no net) -> unconnected-(U2-Pad59)
- U2 pad 6: (no net) -> unconnected-(U2-Pad6)
- U2 pad 60: (no net) -> unconnected-(U2-Pad60)
- U2 pad 61: (no net) -> unconnected-(U2-Pad61)
- U2 pad 62: (no net) -> VCC
- U2 pad 63: (no net) -> unconnected-(U2-Pad63)
- U2 pad 64: (no net) -> unconnected-(U2-Pad64)
- U2 pad 65: (no net) -> unconnected-(U2-Pad65)
- U2 pad 66: (no net) -> unconnected-(U2-Pad66)
- U2 pad 67: (no net) -> unconnected-(U2-Pad67)
- U2 pad 68: (no net) -> unconnected-(U2-Pad68)
- U2 pad 69: (no net) -> unconnected-(U2-Pad69)
- U2 pad 7: (no net) -> unconnected-(U2-Pad7)
- U2 pad 70: (no net) -> unconnected-(U2-Pad70)
- U2 pad 71: (no net) -> unconnected-(U2-Pad71)
- U2 pad 72: (no net) -> unconnected-(U2-Pad72)
- U2 pad 73: (no net) -> unconnected-(U2-Pad73)
- U2 pad 74: (no net) -> unconnected-(U2-Pad74)
- U2 pad 75: (no net) -> unconnected-(U2-Pad75)
- U2 pad 76: (no net) -> unconnected-(U2-Pad76)
- U2 pad 77: (no net) -> unconnected-(U2-Pad77)
- U2 pad 78: (no net) -> unconnected-(U2-Pad78)
- U2 pad 79: (no net) -> unconnected-(U2-Pad79)
- U2 pad 8: (no net) -> unconnected-(U2-Pad8)
- U2 pad 80: (no net) -> unconnected-(U2-Pad80)
- U2 pad 81: (no net) -> VCC
- U2 pad 82: (no net) -> unconnected-(U2-Pad82)
- U2 pad 83: (no net) -> unconnected-(U2-Pad83)
- U2 pad 84: (no net) -> unconnected-(U2-Pad84)
- U2 pad 85: (no net) -> unconnected-(U2-Pad85)
- U2 pad 86: (no net) -> unconnected-(U2-Pad86)
- U2 pad 87: (no net) -> unconnected-(U2-Pad87)
- U2 pad 88: (no net) -> unconnected-(U2-Pad88)
- U2 pad 89: (no net) -> unconnected-(U2-Pad89)
- U2 pad 9: (no net) -> unconnected-(U2-Pad9)
- U2 pad 90: (no net) -> unconnected-(U2-Pad90)
- U2 pad 91: (no net) -> unconnected-(U2-Pad91)
- U2 pad 92: (no net) -> unconnected-(U2-Pad92)
- U2 pad 93: (no net) -> unconnected-(U2-Pad93)
- U2 pad 94: (no net) -> unconnected-(U2-Pad94)
- U2 pad 95: (no net) -> unconnected-(U2-Pad95)
- U2 pad 96: (no net) -> unconnected-(U2-Pad96)
- U2 pad 97: (no net) -> unconnected-(U2-Pad97)
- U2 pad 98: (no net) -> unconnected-(U2-Pad98)
- U2 pad 99: (no net) -> unconnected-(U2-Pad99)
- U3 pad 1: (no net) -> unconnected-(U3-Pad1)
- U3 pad 10: (no net) -> unconnected-(U3-Pad10)
- U3 pad 100: (no net) -> unconnected-(U3-Pad100)
- U3 pad 11: (no net) -> unconnected-(U3-Pad11)
- U3 pad 12: (no net) -> unconnected-(U3-Pad12)
- U3 pad 13: (no net) -> unconnected-(U3-Pad13)
- U3 pad 14: (no net) -> unconnected-(U3-Pad14)
- U3 pad 15: (no net) -> unconnected-(U3-Pad15)
- U3 pad 16: (no net) -> unconnected-(U3-Pad16)
- U3 pad 17: (no net) -> unconnected-(U3-Pad17)
- U3 pad 18: (no net) -> unconnected-(U3-Pad18)
- U3 pad 19: (no net) -> unconnected-(U3-Pad19)
- U3 pad 2: (no net) -> unconnected-(U3-Pad2)
- U3 pad 20: (no net) -> unconnected-(U3-Pad20)
- U3 pad 21: (no net) -> unconnected-(U3-Pad21)
- U3 pad 22: (no net) -> unconnected-(U3-Pad22)
- U3 pad 23: (no net) -> unconnected-(U3-Pad23)
- U3 pad 24: (no net) -> unconnected-(U3-Pad24)
- U3 pad 25: (no net) -> unconnected-(U3-Pad25)
- U3 pad 26: (no net) -> unconnected-(U3-Pad26)
- U3 pad 27: (no net) -> unconnected-(U3-Pad27)
- U3 pad 28: (no net) -> unconnected-(U3-Pad28)
- U3 pad 29: (no net) -> unconnected-(U3-Pad29)
- U3 pad 3: (no net) -> unconnected-(U3-Pad3)
- U3 pad 30: (no net) -> unconnected-(U3-Pad30)
- U3 pad 31: (no net) -> unconnected-(U3-Pad31)
- U3 pad 32: (no net) -> VCC
- U3 pad 33: (no net) -> unconnected-(U3-Pad33)
- U3 pad 34: (no net) -> unconnected-(U3-Pad34)
- U3 pad 35: (no net) -> unconnected-(U3-Pad35)
- U3 pad 36: (no net) -> unconnected-(U3-Pad36)
- U3 pad 37: (no net) -> unconnected-(U3-Pad37)
- U3 pad 38: (no net) -> unconnected-(U3-Pad38)
- U3 pad 39: (no net) -> unconnected-(U3-Pad39)
- U3 pad 4: (no net) -> unconnected-(U3-Pad4)
- U3 pad 40: (no net) -> unconnected-(U3-Pad40)
- U3 pad 41: (no net) -> unconnected-(U3-Pad41)
- U3 pad 42: (no net) -> unconnected-(U3-Pad42)
- U3 pad 43: (no net) -> unconnected-(U3-Pad43)
- U3 pad 44: (no net) -> unconnected-(U3-Pad44)
- U3 pad 45: (no net) -> unconnected-(U3-Pad45)
- U3 pad 46: (no net) -> unconnected-(U3-Pad46)
- U3 pad 47: (no net) -> unconnected-(U3-Pad47)
- U3 pad 48: (no net) -> unconnected-(U3-Pad48)
- U3 pad 49: (no net) -> unconnected-(U3-Pad49)
- U3 pad 5: (no net) -> VCC
- U3 pad 50: (no net) -> unconnected-(U3-Pad50)
- U3 pad 51: (no net) -> unconnected-(U3-Pad51)
- U3 pad 52: (no net) -> unconnected-(U3-Pad52)
- U3 pad 53: (no net) -> unconnected-(U3-Pad53)
- U3 pad 54: (no net) -> unconnected-(U3-Pad54)
- U3 pad 55: (no net) -> unconnected-(U3-Pad55)
- U3 pad 56: (no net) -> unconnected-(U3-Pad56)
- U3 pad 57: (no net) -> unconnected-(U3-Pad57)
- U3 pad 58: (no net) -> unconnected-(U3-Pad58)
- U3 pad 59: (no net) -> VCC
- U3 pad 6: (no net) -> unconnected-(U3-Pad6)
- U3 pad 60: (no net) -> unconnected-(U3-Pad60)
- U3 pad 61: (no net) -> unconnected-(U3-Pad61)
- U3 pad 62: (no net) -> unconnected-(U3-Pad62)
- U3 pad 63: (no net) -> unconnected-(U3-Pad63)
- U3 pad 64: (no net) -> unconnected-(U3-Pad64)
- U3 pad 65: (no net) -> unconnected-(U3-Pad65)
- U3 pad 66: (no net) -> unconnected-(U3-Pad66)
- U3 pad 67: (no net) -> unconnected-(U3-Pad67)
- U3 pad 68: (no net) -> unconnected-(U3-Pad68)
- U3 pad 69: (no net) -> unconnected-(U3-Pad69)
- U3 pad 7: (no net) -> unconnected-(U3-Pad7)
- U3 pad 70: (no net) -> unconnected-(U3-Pad70)
- U3 pad 71: (no net) -> unconnected-(U3-Pad71)
- U3 pad 72: (no net) -> unconnected-(U3-Pad72)
- U3 pad 73: (no net) -> unconnected-(U3-Pad73)
- U3 pad 74: (no net) -> unconnected-(U3-Pad74)
- U3 pad 75: (no net) -> unconnected-(U3-Pad75)
- U3 pad 76: (no net) -> unconnected-(U3-Pad76)
- U3 pad 77: (no net) -> unconnected-(U3-Pad77)
- U3 pad 78: (no net) -> unconnected-(U3-Pad78)
- U3 pad 79: (no net) -> unconnected-(U3-Pad79)
- U3 pad 8: (no net) -> unconnected-(U3-Pad8)
- U3 pad 80: (no net) -> unconnected-(U3-Pad80)
- U3 pad 81: (no net) -> unconnected-(U3-Pad81)
- U3 pad 82: (no net) -> unconnected-(U3-Pad82)
- U3 pad 83: (no net) -> VCC
- U3 pad 84: (no net) -> unconnected-(U3-Pad84)
- U3 pad 85: (no net) -> unconnected-(U3-Pad85)
- U3 pad 86: (no net) -> unconnected-(U3-Pad86)
- U3 pad 87: (no net) -> unconnected-(U3-Pad87)
- U3 pad 88: (no net) -> unconnected-(U3-Pad88)
- U3 pad 89: (no net) -> unconnected-(U3-Pad89)
- U3 pad 9: (no net) -> unconnected-(U3-Pad9)
- U3 pad 90: (no net) -> unconnected-(U3-Pad90)
- U3 pad 91: (no net) -> unconnected-(U3-Pad91)
- U3 pad 92: (no net) -> unconnected-(U3-Pad92)
- U3 pad 93: (no net) -> unconnected-(U3-Pad93)
- U3 pad 94: (no net) -> unconnected-(U3-Pad94)
- U3 pad 95: (no net) -> unconnected-(U3-Pad95)
- U3 pad 96: (no net) -> unconnected-(U3-Pad96)
- U3 pad 97: (no net) -> unconnected-(U3-Pad97)
- U3 pad 98: (no net) -> unconnected-(U3-Pad98)
- U3 pad 99: (no net) -> unconnected-(U3-Pad99)

Commit message: add controller port
Parts:
- added C107: 0.01u, Capacitor_SMD:C_0805_2012Metric, B.Cu at (185.7, 128.3)
- added C35: 330p, Capacitor_SMD:C_0805_2012Metric, B.Cu at (232.4, 146.1)
- added C36: 330p, Capacitor_SMD:C_0805_2012Metric, B.Cu at (232.4, 143.5)
- added C37: 330p, Capacitor_SMD:C_0805_2012Metric, B.Cu at (232.4, 141.0)
- added C38: 330p, Capacitor_SMD:C_0805_2012Metric, B.Cu at (232.4, 138.4)
- added C39: 330p, Capacitor_SMD:C_0805_2012Metric, B.Cu at (232.4, 135.9)
- added C40: 330p, Capacitor_SMD:C_0805_2012Metric, B.Cu at (232.4, 133.3)
- added C41: 330p, Capacitor_SMD:C_0805_2012Metric, B.Cu at (232.4, 130.8)
- added C42: 330p, Capacitor_SMD:C_0805_2012Metric, B.Cu at (232.4, 128.3)
- added C43: 330p, Capacitor_SMD:C_0805_2012Metric, B.Cu at (232.4, 125.7)
- added DA10: D, Package_TO_SOT_SMD:SOT-23, B.Cu at (232.7, 181.7)
- added DA2: D, Package_TO_SOT_SMD:SOT-23, B.Cu at (242.6, 168.8)
- added DA3: D, Package_TO_SOT_SMD:SOT-23, B.Cu at (242.6, 173.3)
- added DA4: D, Package_TO_SOT_SMD:SOT-23, B.Cu at (242.5, 177.7)
- added DA5: D, Package_TO_SOT_SMD:SOT-23, B.Cu at (242.5, 182.1)
- added DA7: D, Package_TO_SOT_SMD:SOT-23, B.Cu at (232.9, 168.8)
- added DA8: D, Package_TO_SOT_SMD:SOT-23, B.Cu at (232.9, 173.3)
- added DA9: D, Package_TO_SOT_SMD:SOT-23, B.Cu at (232.7, 177.2)
- added P2: Conn_2Rows-11Pins, Connector_JST:JST_ZE_B11B-ZESK-D_1x11_P1.50mm_Vertical, F.Cu at (243.5, 142.1)
- added R78: 10k, Resistor_SMD:R_0805_2012Metric, B.Cu at (169.2, 152.4)
- added R80: 10k, Resistor_SMD:R_0805_2012Metric, B.Cu at (164.2, 125.7)
- added R82: 10k, Resistor_SMD:R_0805_2012Metric, B.Cu at (209.0, 151.9)
- added R83: 100, Resistor_SMD:R_0805_2012Metric, B.Cu at (228.2, 146.1)
- added R84: 100, Resistor_SMD:R_0805_2012Metric, B.Cu at (228.2, 143.5)
- added R85: 100, Resistor_SMD:R_0805_2012Metric, B.Cu at (228.2, 141.0)
- added R86: 100, Resistor_SMD:R_0805_2012Metric, B.Cu at (228.2, 138.4)
- added R87: 100, Resistor_SMD:R_0805_2012Metric, B.Cu at (228.2, 135.9)
- added R88: 100, Resistor_SMD:R_0805_2012Metric, B.Cu at (228.2, 133.3)
- added R89: 100, Resistor_SMD:R_0805_2012Metric, B.Cu at (228.2, 130.8)
- added R90: 100, Resistor_SMD:R_0805_2012Metric, B.Cu at (228.2, 128.3)
- added R91: 100, Resistor_SMD:R_0805_2012Metric, B.Cu at (228.2, 125.7)
- added X1: Crystal, Crystal:Crystal_HC49-4H_Vertical, F.Cu at (192.0, 189.2)
- moved DB1 13.0 mm to (108.0, 186.7)
- moved P1 12.0 mm to (153.7, 170.2)
- moved U2 8.62 mm to (214.8, 130.3)
- moved U3 8.62 mm to (184.4, 130.3)
- moved C97 8.62 mm to (216.7, 104.9)
- moved U5 8.14 mm to (188.0, 105.0)
- moved U4 7.49 mm to (216.5, 104.6)
- moved T1 6.42 mm to (83.8, 193.0)
- moved P3 6.11 mm to (105.4, 201.9), turned to 180 degrees
- moved J1 5.24 mm to (72.4, 198.1)
- moved U12 4.02 mm to (114.3, 200.7)
- moved U1 2.84 mm to (210.8, 170.2)
- moved F1 1.83 mm to (109.0, 208.5)
Connections:
- C34 pad 1: Net-(C34-Pad1) -> Net-(P3-Pin_1)
- F1 pad 2: Net-(F1-Pad2) -> Net-(P3-Pin_2)
- P3 pad 1: Net-(F1-Pad2) -> Net-(P3-Pin_1)
- P3 pad 2: Net-(C34-Pad1) -> Net-(P3-Pin_2)
- T1 pad 1: Net-(C30-Pad1) -> Net-(C30-Pad2)
- T1 pad 2: Net-(C30-Pad2) -> Net-(C30-Pad1)
- T1 pad 3: Net-(C31-Pad1) -> Net-(C31-Pad2)
- T1 pad 4: Net-(C31-Pad2) -> Net-(C31-Pad1)
- U1 pad 18: unconnected-(U1-Pad18) -> GND
- U1 pad 47: unconnected-(U1-Pad47) -> GND
- U1 pad 79: unconnected-(U1-Pad79) -> GND
- U1 pad 90: unconnected-(U1-Pad90) -> GND
- U12 pad 1: Net-(C34-Pad1) -> Net-(P3-Pin_1)
- U2 pad 22: unconnected-(U2-Pad22) -> GND
- U2 pad 28: unconnected-(U2-Pad28) -> /VDB0
- U2 pad 29: unconnected-(U2-Pad29) -> /VDB1
- U2 pad 30: unconnected-(U2-Pad30) -> /VDB2
- U2 pad 31: unconnected-(U2-Pad31) -> /VDB3
- U2 pad 32: unconnected-(U2-Pad32) -> /VDB4
- U2 pad 33: unconnected-(U2-Pad33) -> /VDB5
- U2 pad 34: unconnected-(U2-Pad34) -> /VDB6
- U2 pad 35: unconnected-(U2-Pad35) -> /VDB7
- U2 pad 37: unconnected-(U2-Pad37) -> /VDA0
- U2 pad 38: unconnected-(U2-Pad38) -> /VDA1
- U2 pad 39: unconnected-(U2-Pad39) -> /VDA2
- U2 pad 40: unconnected-(U2-Pad40) -> /VDA3
- U2 pad 41: unconnected-(U2-Pad41) -> /VDA4
- U2 pad 42: unconnected-(U2-Pad42) -> /VDA5
- U2 pad 43: unconnected-(U2-Pad43) -> /VDA6
- U2 pad 44: unconnected-(U2-Pad44) -> /VDA7
- U2 pad 45: unconnected-(U2-Pad45) -> GND
- U2 pad 47: unconnected-(U2-Pad47) -> /VA14
- U2 pad 48: unconnected-(U2-Pad48) -> /VAB13
- U2 pad 49: unconnected-(U2-Pad49) -> /VAB12
- U2 pad 50: unconnected-(U2-Pad50) -> /VAB11
- U2 pad 51: unconnected-(U2-Pad51) -> /VAB10
- U2 pad 52: unconnected-(U2-Pad52) -> /VAB9
- U2 pad 53: unconnected-(U2-Pad53) -> /VAB8
- U2 pad 54: unconnected-(U2-Pad54) -> /VAB7
- U2 pad 55: unconnected-(U2-Pad55) -> /VAB6
- U2 pad 56: unconnected-(U2-Pad56) -> /VAB5
- U2 pad 57: unconnected-(U2-Pad57) -> /VAB4
- U2 pad 58: unconnected-(U2-Pad58) -> /VAB3
- U2 pad 59: unconnected-(U2-Pad59) -> /VAB2
- U2 pad 60: unconnected-(U2-Pad60) -> /VAB1
- U2 pad 61: unconnected-(U2-Pad61) -> /VAB0
- U2 pad 63: unconnected-(U2-Pad63) -> /VAA13
- U2 pad 64: unconnected-(U2-Pad64) -> /VAA12
- U2 pad 65: unconnected-(U2-Pad65) -> /VAA11
- U2 pad 66: unconnected-(U2-Pad66) -> /VAA10
- U2 pad 67: unconnected-(U2-Pad67) -> /VAA9
- U2 pad 68: unconnected-(U2-Pad68) -> /VAA8
- U2 pad 69: unconnected-(U2-Pad69) -> /VAA7
- U2 pad 70: unconnected-(U2-Pad70) -> /VAA6
- U2 pad 71: unconnected-(U2-Pad71) -> /VAA5
- U2 pad 72: unconnected-(U2-Pad72) -> /VAA4
- U2 pad 73: unconnected-(U2-Pad73) -> /VAA3
- U2 pad 74: unconnected-(U2-Pad74) -> /VAA2
- U2 pad 75: unconnected-(U2-Pad75) -> /VAA1
- U2 pad 76: unconnected-(U2-Pad76) -> /VAA0
- U2 pad 77: unconnected-(U2-Pad77) -> GND
- U2 pad 96: unconnected-(U2-Pad96) -> GND
- U3 pad 16: unconnected-(U3-Pad16) -> GND
- U3 pad 30: unconnected-(U3-Pad30) -> GND
- U3 pad 35: unconnected-(U3-Pad35) -> GND
- U3 pad 51: unconnected-(U3-Pad51) -> /VDB0
- U3 pad 52: unconnected-(U3-Pad52) -> /VDB1
- U3 pad 53: unconnected-(U3-Pad53) -> /VDB2
- U3 pad 54: unconnected-(U3-Pad54) -> /VDB3
- U3 pad 55: unconnected-(U3-Pad55) -> /VDB4
- U3 pad 56: unconnected-(U3-Pad56) -> /VDB5
- U3 pad 57: unconnected-(U3-Pad57) -> /VDB6
- U3 pad 58: unconnected-(U3-Pad58) -> /VDB7
- U3 pad 60: unconnected-(U3-Pad60) -> /VDA0
- U3 pad 61: unconnected-(U3-Pad61) -> /VDA1
- U3 pad 62: unconnected-(U3-Pad62) -> /VDA2
- U3 pad 63: unconnected-(U3-Pad63) -> /VDA3
- U3 pad 64: unconnected-(U3-Pad64) -> /VDA4
- U3 pad 65: unconnected-(U3-Pad65) -> /VDA5
- U3 pad 66: unconnected-(U3-Pad66) -> /VDA6
- U3 pad 67: unconnected-(U3-Pad67) -> /VDA7
- U3 pad 68: unconnected-(U3-Pad68) -> GND
- U3 pad 69: unconnected-(U3-Pad69) -> /VDB0
- U3 pad 70: unconnected-(U3-Pad70) -> /VDB1
- U3 pad 71: unconnected-(U3-Pad71) -> /VDB2
- U3 pad 72: unconnected-(U3-Pad72) -> /VDB3
- U3 pad 73: unconnected-(U3-Pad73) -> /VDB4
- U3 pad 74: unconnected-(U3-Pad74) -> /VDB5
- U3 pad 75: unconnected-(U3-Pad75) -> /VDB6
- U3 pad 76: unconnected-(U3-Pad76) -> /VDB7
- U3 pad 90: unconnected-(U3-Pad90) -> GND
- U3 pad 91: unconnected-(U3-Pad91) -> GND
- U3 pad 92: unconnected-(U3-Pad92) -> GND
- U3 pad 93: unconnected-(U3-Pad93) -> GND
- U3 pad 94: unconnected-(U3-Pad94) -> VCC
- U3 pad 99: unconnected-(U3-Pad99) -> GND
- U4 pad 1: unconnected-(U4-Pad1) -> /VA14
- U4 pad 10: unconnected-(U4-Pad10) -> /VAB0
- U4 pad 11: /D0 -> /VDB0
- U4 pad 12: /D1 -> /VDB1
- U4 pad 13: /D2 -> /VDB2
- U4 pad 15: /D3 -> /VDB3
- U4 pad 16: /D4 -> /VDB4
- U4 pad 17: /D5 -> /VDB5
- U4 pad 18: /D6 -> /VDB6
- U4 pad 19: /D7 -> /VDB7
- U4 pad 2: unconnected-(U4-Pad2) -> /VAB12
- U4 pad 21: unconnected-(U4-Pad21) -> /VAB10
- U4 pad 23: unconnected-(U4-Pad23) -> /VAB11
- U4 pad 24: unconnected-(U4-Pad24) -> /VAB9
- U4 pad 25: unconnected-(U4-Pad25) -> /VAB8
- U4 pad 26: unconnected-(U4-Pad26) -> /VAB13
- U4 pad 3: unconnected-(U4-Pad3) -> /VAB7
- U4 pad 4: unconnected-(U4-Pad4) -> /VAB6
- U4 pad 5: unconnected-(U4-Pad5) -> /VAB5
- U4 pad 6: unconnected-(U4-Pad6) -> /VAB4
- U4 pad 7: unconnected-(U4-Pad7) -> /VAB3
- U4 pad 8: unconnected-(U4-Pad8) -> /VAB2
- U4 pad 9: unconnected-(U4-Pad9) -> /VAB1
- U5 pad 1: unconnected-(U5-Pad1) -> /VA14
- U5 pad 10: unconnected-(U5-Pad10) -> /VAA0
- U5 pad 11: /D0 -> /VDA0
- U5 pad 12: /D1 -> /VDA1
- U5 pad 13: /D2 -> /VDA2
- U5 pad 15: /D3 -> /VDA3
- U5 pad 16: /D4 -> /VDA4
- U5 pad 17: /D5 -> /VDA5
- U5 pad 18: /D6 -> /VDA6
- U5 pad 19: /D7 -> /VDA7
- U5 pad 2: unconnected-(U5-Pad2) -> /VAA12
- U5 pad 21: unconnected-(U5-Pad21) -> /VAA10
- U5 pad 23: unconnected-(U5-Pad23) -> /VAA11
- U5 pad 24: unconnected-(U5-Pad24) -> /VAA9
- U5 pad 25: unconnected-(U5-Pad25) -> /VAA8
- U5 pad 26: unconnected-(U5-Pad26) -> /VAA13
- U5 pad 3: unconnected-(U5-Pad3) -> /VAA7
- U5 pad 4: unconnected-(U5-Pad4) -> /VAA6
- U5 pad 5: unconnected-(U5-Pad5) -> /VAA5
- U5 pad 6: unconnected-(U5-Pad6) -> /VAA4
- U5 pad 7: unconnected-(U5-Pad7) -> /VAA3
- U5 pad 8: unconnected-(U5-Pad8) -> /VAA2
- U5 pad 9: unconnected-(U5-Pad9) -> /VAA1
Routing:
- net Net-(F1-Pad2): track 23.3 -> 0.00 mm
- net Net-(P3-Pin_2): track 0.00 -> 20.3 mm
- net Net-(C30-Pad2): track 0.00 -> 18.8 mm
- net Net-(C30-Pad1): track 0.00 -> 16.6 mm
- net Net-(P2-Pin_3): track 0.00 -> 16.6 mm
- net Net-(P2-Pin_9): track 0.00 -> 16.2 mm
- net Net-(P2-Pin_5): track 0.00 -> 15.3 mm
- net Net-(P2-Pin_7): track 0.00 -> 15.3 mm
- net Net-(P2-Pin_2): track 0.00 -> 14.6 mm
- net Net-(P2-Pin_10): track 0.00 -> 14.4 mm
- net GND: track 0.00 -> 14.3 mm, vias 0 -> 9
- net Net-(P2-Pin_4): track 0.00 -> 13.8 mm
- net Net-(P2-Pin_8): track 0.00 -> 13.6 mm
- net Net-(P2-Pin_6): track 0.00 -> 12.9 mm
- net Net-(DB1-+): track 12.0 -> 0.00 mm, vias 4 -> 0
- added copper zone on F.Cu, net GND
Other:
- board size 188 x 161.3 mm -> 188 x 158.8 mm
