File: nonSNES.kicad_pcb (KiCad board)
At the start: 4 copper layers, 188 x 158.8 mm, 53 parts, among them J1 Jack-DC, P1 CASSETTE, P2 Conn_2Rows-11Pins, P3 Conn_01x02_Male, T1 L_Coupled, U1 CPU, U12 L7805, U2 PPU1, U3 PPU2, U4 MS62256CL-10FC, U5 MS62256CL-10FC, X1 Crystal

Commit message: add fills
Parts:
- moved DA2 16.5 mm to (228.0, 161.2)
- moved DA3 16.5 mm to (228.0, 165.6)
- moved DA4 16.5 mm to (227.9, 170.0)
- moved DA5 16.5 mm to (227.9, 174.4)
- moved DA7 13.3 mm to (222.0, 161.2)
- moved DA8 13.3 mm to (222.0, 165.6)
- moved DA9 13.3 mm to (221.9, 169.5)
- moved DA10 13.3 mm to (221.9, 174.0)
Other:
- outline, holes or cut-outs redrawn
- copper layers 4 -> 2
Changed lines of the file:
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@@
   (layers
     (0 "F.Cu" signal)
-    (1 "In1.Cu" signal)
-    (2 "In2.Cu" signal)
     (31 "B.Cu" signal)
     (32 "B.Adhes" user "B.Adhesive")
@@
       (layer "F.Mask" (type "Top Solder Mask") (color "Green") (thickness 0.01))
       (layer "F.Cu" (type "copper") (thickness 0.035))
-      (layer "dielectric 1" (type "core") (thickness 1.51) (material "FR4") (epsilon_r 4.5) (loss_tangent 0.02))
-      (layer "In1.Cu" (type "copper") (thickness 0.035))
-      (layer "dielectric 2" (type "prepreg") (thickness 1.51) (material "FR4") (epsilon_r 4.5) (loss_tangent 0.02))
-      (layer "In2.Cu" (type "copper") (thickness 0.035))
-      (layer "dielectric 3" (type "core") (thickness 1.51) (material "FR4") (epsilon_r 4.5) (loss_tangent 0.02))
+      (layer "dielectric 1" (type "core") (thickness 4.6) (material "FR4") (epsilon_r 4.5) (loss_tangent 0.02))
       (layer "B.Cu" (type "copper") (thickness 0.035))
       (layer "B.Mask" (type "Bottom Solder Mask") (color "Green") (thickness 0.01))
@@
     (property "Sheetname" "")
     (attr through_hole)
-    (fp_text reference "P1" (at 2.54 -9.13) (layer "F.SilkS")
+    (fp_text reference "P1" (at -6.35 39.37 270) (layer "F.SilkS")
         (effects (font (size 1 1) (thickness 0.15)))
     )
@@
   )
   (footprint "Package_TO_SOT_SMD:SOT-23" (layer "B.Cu")
-    (at 232.7425 177.226 180)
+    (at 221.9175 169.54 180)
     (descr "SOT, 3 Pin (https://www.jedec.org/system/files/docs/to-236h.pdf variant AB), generated with kicad-footprint-generator ipc_gullwing_generator.py")
     (tags "SOT TO_SOT_SMD")
@@
   )
   (footprint "Package_TO_SOT_SMD:SOT-23" (layer "B.Cu")
-    (at 242.6485 168.844 180)
+    (at 228.0135 161.158 180)
     (descr "SOT, 3 Pin (https://www.jedec.org/system/files/docs/to-236h.pdf variant AB), generated with kicad-footprint-generator ipc_gullwing_generator.py")
     (tags "SOT TO_SOT_SMD")
@@
   )
   (footprint "Package_TO_SOT_SMD:SOT-23" (layer "B.Cu")
-    (at 232.8685 168.844 180)
+    (at 222.0435 161.158 180)
     (descr "SOT, 3 Pin (https://www.jedec.org/system/files/docs/to-236h.pdf variant AB), generated with kicad-footprint-generator ipc_gullwing_generator.py")
     (tags "SOT TO_SOT_SMD")
@@
   )
   (footprint "Package_TO_SOT_SMD:SOT-23" (layer "B.Cu")
-    (at 242.4915 182.118 180)
+    (at 227.8565 174.432 180)
     (descr "SOT, 3 Pin (https://www.jedec.org/system/files/docs/to-236h.pdf variant AB), generated with kicad-footprint-generator ipc_gullwing_generator.py")
     (tags "SOT TO_SOT_SMD")
@@
   )
   (footprint "Package_TO_SOT_SMD:SOT-23" (layer "B.Cu")
-    (at 232.7425 181.676 180)
+    (at 221.9175 173.99 180)
     (descr "SOT, 3 Pin (https://www.jedec.org/system/files/docs/to-236h.pdf variant AB), generated with kicad-footprint-generator ipc_gullwing_generator.py")
     (tags "SOT TO_SOT_SMD")
@@
   )
   (footprint "Package_TO_SOT_SMD:SOT-23" (layer "B.Cu")
-    (at 242.4915 177.668 180)
+    (at 227.8565 169.982 180)
     (descr "SOT, 3 Pin (https://www.jedec.org/system/files/docs/to-236h.pdf variant AB), generated with kicad-footprint-generator ipc_gullwing_generator.py")
     (tags "SOT TO_SOT_SMD")
@@
   )
   (footprint "Package_TO_SOT_SMD:SOT-23" (layer "B.Cu")
-    (at 242.6485 173.294 180)
+    (at 228.0135 165.608 180)
     (descr "SOT, 3 Pin (https://www.jedec.org/system/files/docs/to-236h.pdf variant AB), generated with kicad-footprint-generator ipc_gullwing_generator.py")
     (tags "SOT TO_SOT_SMD")
@@
   )
   (footprint "Package_TO_SOT_SMD:SOT-23" (layer "B.Cu")
-    (at 232.8685 173.294 180)
+    (at 222.0435 165.608 180)
     (descr "SOT, 3 Pin (https://www.jedec.org/system/files/docs/to-236h.pdf variant AB), generated with kicad-footprint-generator ipc_gullwing_generator.py")
     (tags "SOT TO_SOT_SMD")
@@
     )
   )
+  (gr_circle (center 127 209.55) (end 129.54 209.55)
+    (stroke (width 0.15) (type solid)) (fill solid) (layer "B.Mask"))
+  (gr_circle (center 78.74 166.37) (end 81.28 166.37)
+    (stroke (width 0.15) (type solid)) (fill solid) (layer "B.Mask"))
+  (gr_circle (center 92.71 209.55) (end 95.25 209.55)
+    (stroke (width 0.15) (type solid)) (fill solid) (layer "B.Mask"))
+  (gr_circle (center 96.52 172.72) (end 99.06 172.72)
+    (stroke (width 0.15) (type solid)) (fill solid) (layer "B.Mask"))
+  (gr_circle (center 109.22 55.88) (end 111.76 55.88)
+    (stroke (width 0.15) (type solid)) (fill solid) (layer "B.Mask"))
   (gr_line (start 126.365 58.42) (end 126.365 53.34)
     (stroke (width 0.1) (type solid)) (layer "Edge.Cuts"))
+  (gr_circle (center 248.92 209.55) (end 248.92 208.28)
+    (stroke (width 0.1) (type default)) (fill none) (layer "Edge.Cuts"))
   (gr_line (start 168.275 53.34) (end 168.275 68.58)
     (stroke (width 0.1) (type solid)) (layer "Edge.Cuts"))
@@
   (gr_line (start 226.06 196.85) (end 236.22 196.85)
     (stroke (width 0.1) (type solid)) (layer "Edge.Cuts"))
+  (gr_circle (center 67.31 67.31) (end 67.31 66.04)
+    (stroke (width 0.1) (type default)) (fill none) (layer "Edge.Cuts"))
   (gr_line (start 104.14 205.74) (end 114.3 205.74)
     (stroke (width 0.1) (type solid)) (layer "Edge.Cuts"))
+  (gr_circle (center 248.92 55.88) (end 247.65 54.61)
+    (stroke (width 0.1) (type default)) (fill none) (layer "Edge.Cuts"))
+  (gr_circle (center 92.71 209.55) (end 92.71 208.28)
+    (stroke (width 0.1) (type default)) (fill none) (layer "Edge.Cuts"))
   (gr_line (start 145.415 53.34) (end 145.415 66.04)
     (stroke (width 0.1) (type solid)) (layer "Edge.Cuts"))
+  (gr_circle (center 140.97 198.12) (end 140.97 196.85)
+    (stroke (width 0.1) (type default)) (fill none) (layer "Edge.Cuts"))
   (gr_line (start 72.39 60.96) (end 72.39 53.34)
     (stroke (width 0.1) (type solid)) (layer "Edge.Cuts"))
@@
   (gr_line (start 63.5 120.65) (end 69.85 120.65)
     (stroke (width 0.1) (type solid)) (layer "Edge.Cuts"))
+  (gr_circle (center 73.66 190.5) (end 73.66 189.23)
+    (stroke (width 0.1) (type default)) (fill none) (layer "Edge.Cuts"))
+  (gr_circle (center 140.97 208.28) (end 140.97 207.01)
+    (stroke (width 0.1) (type default)) (fill none) (layer "Edge.Cuts"))
   (gr_line (start 104.14 212.09) (end 78.74 212.09)
     (stroke (width 0.1) (type solid)) (layer "Edge.Cuts"))
@@
   (gr_line (start 191.77 212.09) (end 191.77 196.85)
     (stroke (width 0.1) (type solid)) (layer "Edge.Cuts"))
+  (gr_circle (center 210.82 199.39) (end 210.82 198.12)
+    (stroke (width 0.1) (type default)) (fill none) (layer "Edge.Cuts"))
   (gr_line (start 201.93 212.09) (end 226.06 212.09)
     (stroke (width 0.1) (type solid)) (layer "Edge.Cuts"))
@@
   (gr_line (start 182.88 212.09) (end 191.77 212.09)
     (stroke (width 0.1) (type solid)) (layer "Edge.Cuts"))
+  (gr_circle (center 213.36 67.31) (end 213.36 66.04)
+    (stroke (width 0.1) (type default)) (fill none) (layer "Edge.Cuts"))
   (gr_line (start 201.93 196.85) (end 201.93 212.09)
     (stroke (width 0.1) (type solid)) (layer "Edge.Cuts"))
@@
   (gr_line (start 191.77 196.85) (end 201.93 196.85)
     (stroke (width 0.1) (type solid)) (layer "Edge.Cuts"))
+  (gr_circle (center 74.93 55.88) (end 74.93 54.61)
+    (stroke (width 0.1) (type default)) (fill none) (layer "Edge.Cuts"))
+  (gr_circle (center 127 209.55) (end 127 208.28)
+    (stroke (width 0.1) (type default)) (fill none) (layer "Edge.Cuts"))
   (gr_text "黒" (at 109.22 200.66) (layer "F.SilkS")
     (effects (font (size 2 1) (thickness 0.15)))
@@
         (xy 121.92 212.09)
         (xy 121.92 194.31)
+        (xy 143.51 194.31)
+        (xy 143.51 179.07)
+        (xy 165.1 179.07)
+        (xy 165.1 194.31)
         (xy 233.68 194.31)
         (xy 233.68 71.12)
@@
       )
     )
+  )
+  (zone (net 0) (net_name "") (layer "B.Mask") (hatch edge 0.5)
+    (connect_pads (clearance 0))
+    (min_thickness 0.25) (filled_areas_thickness no)
+    (keepout (tracks not_allowed) (vias not_allowed) (pads not_allowed) (copperpour allowed) (footprints allowed))
+    (fill (thermal_gap 0.5) (thermal_bridge_width 0.5))
+    (polygon
+      (pts
+        (xy 251.46 162.56)
+        (xy 238.76 162.56)
+        (xy 238.76 181.61)
+        (xy 251.46 181.61)
+      )
+    )
+  )
+  (zone (net 0) (net_name "") (layer "F.Mask") (hatch edge 0.5)
+    (connect_pads (clearance 0))
+    (min_thickness 0.25) (filled_areas_thickness no)
+    (keepout (tracks not_allowed) (vias not_allowed) (pads not_allowed) (copperpour allowed) (footprints allowed))
+    (fill (thermal_gap 0.5) (thermal_bridge_width 0.5))
+    (polygon
+      (pts
+        (xy 143.51 179.07)
+        (xy 158.75 179.07)
+        (xy 158.75 212.09)
+        (xy 143.51 212.09)
+      )
+    )

Commit message: more copper
Parts:
- moved C95 7.73 mm to (190.5, 105.4)
- moved U4 2.54 mm to (219.1, 104.6)
- moved U5 0.63 mm to (188.6, 105.0)
Other:
- outline, holes or cut-outs redrawn
- board text added: "1992"
Changed lines of the file:
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@@
   )
   (footprint "Package_SO:SOIC-28W_7.5x17.9mm_P1.27mm" (layer "F.Cu")
-    (at 187.96 104.98 90)
+    (at 188.595 104.98 90)
     (descr "SOIC, 28 Pin (JEDEC MS-013AE, https://www.analog.com/media/en/package-pcb-resources/package/35833120341221rw_28.pdf), generated with kicad-footprint-generator ipc_gullwing_generator.py")
     (tags "SOIC SO")
@@
     (property "ki_keywords" "RAM SRAM CMOS MEMORY")
     (attr smd)
-    (fp_text reference "U5" (at 0 -9.9 90) (layer "F.SilkS")
+    (fp_text reference "U5" (at 8.46 -1.905 180) (layer "F.SilkS")
         (effects (font (size 1 1) (thickness 0.15)))
     )
@@
     (property "ki_keywords" "DC power barrel jack connector")
     (attr through_hole)
-    (fp_text reference "J1" (at 0 -6.35 unlocked) (layer "F.SilkS")
+    (fp_text reference "J1" (at 7.62 -7.62 90 unlocked) (layer "F.SilkS")
         (effects (font (size 1 1) (thickness 0.15)))
     )
@@
     (property "ki_keywords" "inductor choke coil reactor magnetic coupled")
     (attr smd)
-    (fp_text reference "T1" (at 0 -4 90) (layer "F.SilkS")
+    (fp_text reference "T1" (at -0.06 5.08 180) (layer "F.SilkS")
         (effects (font (size 1 1) (thickness 0.15)))
     )
@@
   )
   (footprint "Package_SO:SOIC-28W_7.5x17.9mm_P1.27mm" (layer "F.Cu")
-    (at 216.535 104.57 90)
+    (at 219.075 104.57 90)
     (descr "SOIC, 28 Pin (JEDEC MS-013AE, https://www.analog.com/media/en/package-pcb-resources/package/35833120341221rw_28.pdf), generated with kicad-footprint-generator ipc_gullwing_generator.py")
     (tags "SOIC SO")
@@
     (property "ki_keywords" "RAM SRAM CMOS MEMORY")
     (attr smd)
-    (fp_text reference "U4" (at 0 -9.9 90) (layer "F.SilkS")
+    (fp_text reference "U4" (at 8.05 -3.175 180) (layer "F.SilkS")
         (effects (font (size 1 1) (thickness 0.15)))
     )
@@
   )
   (footprint "Capacitor_SMD:C_0805_2012Metric" (layer "B.Cu")
-    (at 191.77 97.79 90)
+    (at 190.5 105.41 90)
     (descr "Capacitor SMD 0805 (2012 Metric), square (rectangular) end terminal, IPC_7351 nominal, (Body size source: IPC-SM-782 page 76, https://www.pcb-3d.com/wordpress/wp-content/uploads/ipc-sm-782a_amendment_1_and_2.pdf, https://docs.google.com/spreadsheets/d/1BsfQQcO9C6DZCsRaXUlFlo91Tg2WpOkGARC1WS5S8t0/edit?usp=sharing), generated with kicad-footprint-generator")
     (tags "capacitor")
@@
   (gr_line (start 63.5 120.65) (end 69.85 120.65)
     (stroke (width 0.1) (type solid)) (layer "Edge.Cuts"))
-  (gr_circle (center 73.66 190.5) (end 73.66 189.23)
+  (gr_circle (center 73.66 190.5) (end 73.66 187.96)
     (stroke (width 0.1) (type default)) (fill none) (layer "Edge.Cuts"))
   (gr_circle (center 140.97 208.28) (end 140.97 207.01)
@@
     (effects (font (size 2 1) (thickness 0.15)))
   )
-  (gr_text "SNSP-CPU-01" (at 181.61 74.93) (layer "F.SilkS")
-    (effects (font (size 1 1) (thickness 0.15)))
+  (gr_text "1992" (at 173.99 76.2) (layer "F.SilkS")
+    (effects (font (size 2 2) (thickness 0.15)) (justify left bottom))
+  )
+  (gr_text "SNSP-CPU-01" (at 181.61 78.74) (layer "F.SilkS")
+    (effects (font (size 2 2) (thickness 0.15)))
   )
   (gr_text "赤" (at 99.06 200.66) (layer "F.SilkS")
@@
         (xy 143.51 77.47)
         (xy 130.81 64.77)
+        (xy 85.09 64.77)
+        (xy 85.09 71.12)
+        (xy 68.58 189.23)
+        (xy 63.5 189.23)
         (xy 63.5 64.77)
         (xy 63.5 53.34)
@@
     (connect_pads (clearance 0))
     (min_thickness 0.25) (filled_areas_thickness no)
+    (keepout (tracks not_allowed) (vias not_allowed) (pads not_allowed) (copperpour allowed) (footprints allowed))
+    (fill (thermal_gap 0.5) (thermal_bridge_width 0.5))
+    (polygon
+      (pts
+        (xy 143.51 88.9)
+        (xy 158.75 88.9)
+        (xy 158.75 53.34)
+        (xy 143.51 53.34)
+      )
+    )
+  )
+  (zone (net 0) (net_name "") (layer "F.Mask") (hatch edge 0.5)
+    (connect_pads (clearance 0))
+    (min_thickness 0.25) (filled_areas_thickness no)
     (fill yes (thermal_gap 0.5) (thermal_bridge_width 0.5))
     (polygon
@@
       )
     )
+  )
+  (zone (net 0) (net_name "") (layer "F.Mask") (hatch edge 0.5)
+    (connect_pads (clearance 0))
+    (min_thickness 0.25) (filled_areas_thickness no)
+    (keepout (tracks not_allowed) (vias not_allowed) (pads not_allowed) (copperpour allowed) (footprints allowed))
+    (fill (thermal_gap 0.5) (thermal_bridge_width 0.5))
+    (polygon
+      (pts
+        (xy 72.39 53.34)
+        (xy 118.11 53.34)
+        (xy 118.11 64.77)
+        (xy 72.39 64.77)
+      )
+    )
