File: nonSNES.kicad_pcb (KiCad board)
At the start: 2 copper layers, 188 x 158.8 mm, 53 parts, among them J1 Jack-DC, P1 CASSETTE, P2 Conn_2Rows-11Pins, P3 Conn_01x02_Male, T1 L_Coupled, U1 CPU, U12 L7805, U2 PPU1, U3 PPU2, U4 MS62256CL-10FC, U5 MS62256CL-10FC, X1 Crystal

Commit message: back end
Parts:
- moved DB1 1.80 mm to (106.7, 188.0)
Other:
- outline, holes or cut-outs redrawn
Changed lines of the file:
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@@
   )
   (footprint "SNES_Library:FullBridgeRectifier" (layer "F.Cu")
-    (at 107.95 186.69)
+    (at 106.68 187.96)
     (property "Sheetfile" "nonSNES.kicad_sch")
     (property "Sheetname" "")
@@
     )
   )
-  (gr_circle (center 127 209.55) (end 129.54 209.55)
-    (stroke (width 0.15) (type solid)) (fill solid) (layer "B.Mask"))
-  (gr_circle (center 78.74 166.37) (end 81.28 166.37)
+  (gr_circle (center 72.39 166.37) (end 76.2 166.37)
     (stroke (width 0.15) (type solid)) (fill solid) (layer "B.Mask"))
   (gr_circle (center 92.71 209.55) (end 95.25 209.55)
     (stroke (width 0.15) (type solid)) (fill solid) (layer "B.Mask"))
-  (gr_circle (center 96.52 172.72) (end 99.06 172.72)
-    (stroke (width 0.15) (type solid)) (fill solid) (layer "B.Mask"))
   (gr_circle (center 109.22 55.88) (end 111.76 55.88)
     (stroke (width 0.15) (type solid)) (fill solid) (layer "B.Mask"))
   (gr_line (start 126.365 58.42) (end 126.365 53.34)
     (stroke (width 0.1) (type solid)) (layer "Edge.Cuts"))
+  (gr_circle (center 72.39 166.37) (end 72.39 163.83)
+    (stroke (width 0.1) (type default)) (fill none) (layer "Edge.Cuts"))
   (gr_circle (center 248.92 209.55) (end 248.92 208.28)
     (stroke (width 0.1) (type default)) (fill none) (layer "Edge.Cuts"))
@@
   (gr_line (start 226.06 196.85) (end 236.22 196.85)
     (stroke (width 0.1) (type solid)) (layer "Edge.Cuts"))
-  (gr_circle (center 67.31 67.31) (end 67.31 66.04)
+  (gr_circle (center 68.58 72.39) (end 68.58 71.12)
     (stroke (width 0.1) (type default)) (fill none) (layer "Edge.Cuts"))
   (gr_line (start 104.14 205.74) (end 114.3 205.74)
@@
   (gr_line (start 145.415 53.34) (end 145.415 66.04)
     (stroke (width 0.1) (type solid)) (layer "Edge.Cuts"))
-  (gr_circle (center 140.97 198.12) (end 140.97 196.85)
+  (gr_circle (center 138.43 198.12) (end 138.43 196.85)
     (stroke (width 0.1) (type default)) (fill none) (layer "Edge.Cuts"))
   (gr_line (start 72.39 60.96) (end 72.39 53.34)
@@
   (gr_line (start 126.365 53.34) (end 145.415 53.34)
     (stroke (width 0.1) (type solid)) (layer "Edge.Cuts"))
+  (gr_circle (center 68.58 137.16) (end 68.58 135.89)
+    (stroke (width 0.1) (type default)) (fill none) (layer "Edge.Cuts"))
   (gr_line (start 63.5 110.49) (end 63.5 60.96)
     (stroke (width 0.1) (type solid)) (layer "Edge.Cuts"))
@@
   (gr_line (start 63.5 120.65) (end 69.85 120.65)
     (stroke (width 0.1) (type solid)) (layer "Edge.Cuts"))
-  (gr_circle (center 73.66 190.5) (end 73.66 187.96)
+  (gr_circle (center 72.39 190.5) (end 72.39 187.96)
     (stroke (width 0.1) (type default)) (fill none) (layer "Edge.Cuts"))
-  (gr_circle (center 140.97 208.28) (end 140.97 207.01)
+  (gr_circle (center 138.43 208.28) (end 138.43 207.01)
     (stroke (width 0.1) (type default)) (fill none) (layer "Edge.Cuts"))
   (gr_line (start 104.14 212.09) (end 78.74 212.09)
@@
   (gr_line (start 78.74 212.09) (end 78.74 204.47)
     (stroke (width 0.1) (type solid)) (layer "Edge.Cuts"))
+  (gr_circle (center 68.58 129.54) (end 68.58 128.27)
+    (stroke (width 0.1) (type default)) (fill none) (layer "Edge.Cuts"))
   (gr_line (start 251.46 212.09) (end 251.46 53.34)
     (stroke (width 0.1) (type solid)) (layer "Edge.Cuts"))
@@
   (gr_line (start 146.05 212.09) (end 146.05 198.12)
     (stroke (width 0.1) (type solid)) (layer "Edge.Cuts"))
+  (gr_circle (center 71.12 124.46) (end 71.12 123.19)
+    (stroke (width 0.1) (type default)) (fill none) (layer "Edge.Cuts"))
   (gr_line (start 114.3 205.74) (end 114.3 212.09)
     (stroke (width 0.1) (type solid)) (layer "Edge.Cuts"))
   (gr_line (start 191.77 196.85) (end 201.93 196.85)
     (stroke (width 0.1) (type solid)) (layer "Edge.Cuts"))
-  (gr_circle (center 74.93 55.88) (end 74.93 54.61)
+  (gr_circle (center 76.2 57.15) (end 76.2 55.88)
     (stroke (width 0.1) (type default)) (fill none) (layer "Edge.Cuts"))
-  (gr_circle (center 127 209.55) (end 127 208.28)
+  (gr_circle (center 125.73 209.55) (end 125.73 208.28)
     (stroke (width 0.1) (type default)) (fill none) (layer "Edge.Cuts"))
   (gr_text "黒" (at 109.22 200.66) (layer "F.SilkS")
@@
         (xy 143.51 77.47)
         (xy 130.81 64.77)
-        (xy 85.09 64.77)
-        (xy 85.09 71.12)
-        (xy 68.58 189.23)
+        (xy 83.82 64.77)
+        (xy 83.82 71.12)
+        (xy 83.82 181.61)
+        (xy 73.66 181.61)
+        (xy 73.66 189.23)
         (xy 63.5 189.23)
         (xy 63.5 64.77)

Commit message: fix drc
Parts:
- C34, C81: moved to B.Cu
- moved C31 21.0 mm to (83.8, 192.4)
- moved C81 3.82 mm to (126.4, 188.9), turned to 90 degrees
- moved C34 2.54 mm to (120.7, 189.2), turned to 90 degrees
- moved C30 2.03 mm to (83.5, 195.6)
- moved DB1 0.64 mm to (106.0, 188.0)
- moved U5 0.63 mm to (189.2, 105.0)
Other:
- outline, holes or cut-outs redrawn

Commit message: fix mask area
Parts:
- moved C35 2.62 mm to (233.0, 143.5)
- moved C38 2.62 mm to (233.0, 135.9)
- moved R83 2.62 mm to (228.9, 143.5)
- moved R86 2.62 mm to (228.9, 135.9)
- moved C42 2.62 mm to (233.0, 125.7)
- moved C43 2.62 mm to (233.0, 123.2)
- moved R90 2.62 mm to (228.9, 125.7)
- moved R91 2.62 mm to (228.9, 123.2)
- moved C36 2.62 mm to (233.0, 141.0)
- moved C37 2.62 mm to (233.0, 138.4)
- moved C39 2.62 mm to (233.0, 133.3)
- moved C40 2.62 mm to (233.0, 130.8)
- moved C41 2.62 mm to (233.0, 128.3)
- moved P2 2.62 mm to (244.2, 139.6)
- moved R84 2.62 mm to (228.9, 141.0)
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Other:
- outline, holes or cut-outs redrawn

Commit message: masks
Parts:
- moved C81 1.80 mm to (125.1, 190.2)
- moved DB1 1.27 mm to (107.3, 188.0)
- moved C34 1.15 mm to (120.0, 190.2)
Other:
- outline, holes or cut-outs redrawn
- board text added: "G"
- board text added: "I"
- board text added: "O"
Changed lines of the file:
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@@
   )
   (footprint "SNES_Library:FullBridgeRectifier" (layer "F.Cu")
-    (at 106.045 187.96)
+    (at 107.315 187.96)
     (property "Sheetfile" "nonSNES.kicad_sch")
     (property "Sheetname" "")
@@
   )
   (footprint "Capacitor_SMD:C_0805_2012Metric" (layer "B.Cu")
-    (at 120.65 189.23 90)
+    (at 120.015 190.185 90)
     (descr "Capacitor SMD 0805 (2012 Metric), square (rectangular) end terminal, IPC_7351 nominal, (Body size source: IPC-SM-782 page 76, https://www.pcb-3d.com/wordpress/wp-content/uploads/ipc-sm-782a_amendment_1_and_2.pdf, https://docs.google.com/spreadsheets/d/1BsfQQcO9C6DZCsRaXUlFlo91Tg2WpOkGARC1WS5S8t0/edit?usp=sharing), generated with kicad-footprint-generator")
     (tags "capacitor")
@@
   )
   (footprint "Capacitor_SMD:C_0805_2012Metric" (layer "B.Cu")
-    (at 126.365 188.915 90)
+    (at 125.095 190.185 90)
     (descr "Capacitor SMD 0805 (2012 Metric), square (rectangular) end terminal, IPC_7351 nominal, (Body size source: IPC-SM-782 page 76, https://www.pcb-3d.com/wordpress/wp-content/uploads/ipc-sm-782a_amendment_1_and_2.pdf, https://docs.google.com/spreadsheets/d/1BsfQQcO9C6DZCsRaXUlFlo91Tg2WpOkGARC1WS5S8t0/edit?usp=sharing), generated with kicad-footprint-generator")
     (tags "capacitor")
@@
     )
   )
-  (gr_circle (center 73.66 158.115) (end 77.47 158.115)
+  (gr_circle (center 73.025 158.75) (end 76.835 158.75)
     (stroke (width 0.15) (type solid)) (fill solid) (layer "B.Mask"))
   (gr_circle (center 92.71 209.55) (end 95.25 209.55)
     (stroke (width 0.15) (type solid)) (fill solid) (layer "B.Mask"))
-  (gr_circle (center 109.22 55.88) (end 111.76 55.88)
+  (gr_circle (center 107.315 57.15) (end 111.125 57.15)
+    (stroke (width 0.15) (type solid)) (fill solid) (layer "B.Mask"))
+  (gr_circle (center 125.73 208.915) (end 128.905 208.915)
     (stroke (width 0.15) (type solid)) (fill solid) (layer "B.Mask"))
   (gr_line (start 126.365 58.42) (end 126.365 53.34)
     (stroke (width 0.1) (type solid)) (layer "Edge.Cuts"))
-  (gr_circle (center 73.66 158.115) (end 73.66 155.575)
+  (gr_circle (center 73.025 158.75) (end 73.025 156.845)
     (stroke (width 0.1) (type default)) (fill none) (layer "Edge.Cuts"))
   (gr_circle (center 247.015 208.28) (end 247.015 207.01)
@@
   (gr_line (start 145.415 53.34) (end 145.415 66.04)
     (stroke (width 0.1) (type solid)) (layer "Edge.Cuts"))
-  (gr_circle (center 109.22 55.88) (end 109.22 54.61)
+  (gr_circle (center 107.315 57.15) (end 107.315 55.245)
     (stroke (width 0.1) (type default)) (fill none) (layer "Edge.Cuts"))
-  (gr_circle (center 242.57 186.055) (end 242.57 184.785)
+  (gr_circle (center 241.935 182.88) (end 241.935 181.61)
     (stroke (width 0.1) (type default)) (fill none) (layer "Edge.Cuts"))
-  (gr_circle (center 138.43 198.12) (end 138.43 196.85)
+  (gr_circle (center 137.795 198.12) (end 137.795 196.85)
     (stroke (width 0.1) (type default)) (fill none) (layer "Edge.Cuts"))
-  (gr_circle (center 138.43 63.5) (end 138.43 62.23)
+  (gr_circle (center 136.525 67.31) (end 136.525 66.04)
     (stroke (width 0.1) (type default)) (fill none) (layer "Edge.Cuts"))
   (gr_line (start 72.39 60.96) (end 72.39 53.34)
@@
   (gr_circle (center 72.39 189.865) (end 72.39 187.325)
     (stroke (width 0.1) (type default)) (fill none) (layer "Edge.Cuts"))
-  (gr_circle (center 138.43 208.28) (end 138.43 207.01)
+  (gr_circle (center 137.795 208.28) (end 137.795 207.01)
     (stroke (width 0.1) (type default)) (fill none) (layer "Edge.Cuts"))
   (gr_line (start 104.14 212.09) (end 78.74 212.09)
@@
   (gr_line (start 191.77 196.85) (end 201.93 196.85)
     (stroke (width 0.1) (type solid)) (layer "Edge.Cuts"))
-  (gr_circle (center 125.73 209.55) (end 125.73 208.28)
+  (gr_circle (center 125.73 208.915) (end 125.73 207.645)
     (stroke (width 0.1) (type default)) (fill none) (layer "Edge.Cuts"))
+  (gr_text "O" (at 120.65 205.105) (layer "B.SilkS")
+    (effects (font (size 2 2) (thickness 0.15)) (justify left bottom mirror))
+  )
+  (gr_text "G" (at 118.11 205.105) (layer "B.SilkS")
+    (effects (font (size 2 2) (thickness 0.15)) (justify left bottom mirror))
+  )
+  (gr_text "I" (at 114.935 205.105) (layer "B.SilkS")
+    (effects (font (size 2 2) (thickness 0.15)) (justify left bottom mirror))
+  )
   (gr_text "黒" (at 109.22 201.295) (layer "F.SilkS")
     (effects (font (size 2 1) (thickness 0.15)))
@@
     )
   )
+  (zone (net 0) (net_name "") (layer "B.Mask") (hatch edge 0.5)
+    (connect_pads (clearance 0))
+    (min_thickness 0.25) (filled_areas_thickness no)
+    (fill yes (thermal_gap 0.5) (thermal_bridge_width 0.5))
+    (polygon
+      (pts
+        (xy 238.76 164.465)
+        (xy 251.46 164.465)
+        (xy 251.46 177.8)
+        (xy 238.76 177.8)
+      )
+    )
+  )
+  (zone (net 0) (net_name "") (layer "B.Mask") (hatch edge 0.5)
+    (connect_pads (clearance 0))
+    (min_thickness 0.25) (filled_areas_thickness no)
+    (fill yes (thermal_gap 0.5) (thermal_bridge_width 0.5))
+    (polygon
+      (pts
+        (xy 69.85 101.6)
+        (xy 63.5 101.6)
+        (xy 63.5 90.17)
+        (xy 69.85 90.17)
+      )
+    )
+  )
   (zone (net 0) (net_name "") (layer "F.Mask") (hatch edge 0.5)
     (connect_pads (clearance 0))
@@
       )
     )
-  )
-  (zone (net 0) (net_name "") (layer "Edge.Cuts") (hatch edge 0.5)
-    (connect_pads (clearance 0))
-    (min_thickness 0.25) (filled_areas_thickness no)
-    (fill yes (thermal_gap 0.5) (thermal_bridge_width 0.5))
-    (polygon
-      (pts
-        (xy 251.46 162.56)
-        (xy 238.76 162.56)
-        (xy 238.76 181.61)
-        (xy 251.46 181.61)
-      )
-    )

Commit message: bottom copper fill
Parts:
- moved C34 1.42 mm to (119.4, 191.5)
- moved C81 1.42 mm to (124.5, 191.5)
- moved C30 1.31 mm to (83.8, 194.3)
- moved C31 1.27 mm to (83.8, 191.1)
Routing:
- added copper zone on B.Cu, net GND
Other:
- outline, holes or cut-outs redrawn
Changed lines of the file:
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@@
   )
   (footprint "Capacitor_SMD:C_0805_2012Metric" (layer "B.Cu")
-    (at 120.015 190.185 90)
+    (at 119.38 191.455 90)
     (descr "Capacitor SMD 0805 (2012 Metric), square (rectangular) end terminal, IPC_7351 nominal, (Body size source: IPC-SM-782 page 76, https://www.pcb-3d.com/wordpress/wp-content/uploads/ipc-sm-782a_amendment_1_and_2.pdf, https://docs.google.com/spreadsheets/d/1BsfQQcO9C6DZCsRaXUlFlo91Tg2WpOkGARC1WS5S8t0/edit?usp=sharing), generated with kicad-footprint-generator")
     (tags "capacitor")
@@
   )
   (footprint "Capacitor_SMD:C_0805_2012Metric" (layer "B.Cu")
-    (at 125.095 190.185 90)
+    (at 124.46 191.455 90)
     (descr "Capacitor SMD 0805 (2012 Metric), square (rectangular) end terminal, IPC_7351 nominal, (Body size source: IPC-SM-782 page 76, https://www.pcb-3d.com/wordpress/wp-content/uploads/ipc-sm-782a_amendment_1_and_2.pdf, https://docs.google.com/spreadsheets/d/1BsfQQcO9C6DZCsRaXUlFlo91Tg2WpOkGARC1WS5S8t0/edit?usp=sharing), generated with kicad-footprint-generator")
     (tags "capacitor")
@@
   )
   (footprint "Capacitor_SMD:C_0805_2012Metric" (layer "B.Cu")
-    (at 83.5 195.58)
+    (at 83.82 194.31)
     (descr "Capacitor SMD 0805 (2012 Metric), square (rectangular) end terminal, IPC_7351 nominal, (Body size source: IPC-SM-782 page 76, https://www.pcb-3d.com/wordpress/wp-content/uploads/ipc-sm-782a_amendment_1_and_2.pdf, https://docs.google.com/spreadsheets/d/1BsfQQcO9C6DZCsRaXUlFlo91Tg2WpOkGARC1WS5S8t0/edit?usp=sharing), generated with kicad-footprint-generator")
     (tags "capacitor")
@@
   )
   (footprint "Capacitor_SMD:C_0805_2012Metric" (layer "B.Cu")
-    (at 83.82 192.405 180)
+    (at 83.82 191.135 180)
     (descr "Capacitor SMD 0805 (2012 Metric), square (rectangular) end terminal, IPC_7351 nominal, (Body size source: IPC-SM-782 page 76, https://www.pcb-3d.com/wordpress/wp-content/uploads/ipc-sm-782a_amendment_1_and_2.pdf, https://docs.google.com/spreadsheets/d/1BsfQQcO9C6DZCsRaXUlFlo91Tg2WpOkGARC1WS5S8t0/edit?usp=sharing), generated with kicad-footprint-generator")
     (tags "capacitor")
@@
   (gr_circle (center 73.025 158.75) (end 76.835 158.75)
     (stroke (width 0.15) (type solid)) (fill solid) (layer "B.Mask"))
-  (gr_circle (center 92.71 209.55) (end 95.25 209.55)
+  (gr_rect (start 238.76 160.655) (end 251.46 176.53)
+    (stroke (width 0.15) (type solid)) (fill solid) (layer "B.Mask"))
+  (gr_rect (start 69.85 90.17) (end 63.5 102.87)
+    (stroke (width 0.15) (type solid)) (fill solid) (layer "B.Mask"))
+  (gr_circle (center 92.71 209.55) (end 95.885 209.55)
     (stroke (width 0.15) (type solid)) (fill solid) (layer "B.Mask"))
   (gr_circle (center 107.315 57.15) (end 111.125 57.15)
     (stroke (width 0.15) (type solid)) (fill solid) (layer "B.Mask"))
-  (gr_circle (center 125.73 208.915) (end 128.905 208.915)
+  (gr_circle (center 125.73 208.915) (end 129.54 208.915)
     (stroke (width 0.15) (type solid)) (fill solid) (layer "B.Mask"))
   (gr_line (start 126.365 58.42) (end 126.365 53.34)
@@
   (gr_arc (start 76.2 59.69) (mid 74.295 57.785) (end 76.2 55.88)
     (stroke (width 0.1) (type default)) (layer "Edge.Cuts"))
-  (gr_circle (center 69.85 137.16) (end 69.85 135.255)
+  (gr_circle (center 70.485 137.16) (end 70.485 135.89)
     (stroke (width 0.1) (type default)) (fill none) (layer "Edge.Cuts"))
   (gr_line (start 63.5 110.49) (end 63.5 60.96)
@@
   (gr_line (start 78.74 212.09) (end 78.74 204.47)
     (stroke (width 0.1) (type solid)) (layer "Edge.Cuts"))
-  (gr_circle (center 69.85 149.225) (end 69.85 147.32)
+  (gr_circle (center 70.485 149.86) (end 70.485 148.59)
     (stroke (width 0.1) (type default)) (fill none) (layer "Edge.Cuts"))
   (gr_line (start 251.46 212.09) (end 251.46 53.34)
@@
     )
   )
-  (zone (net 0) (net_name "") (layer "B.Mask") (hatch edge 0.5)
+  (zone (net 245) (net_name "GND") (layer "B.Cu") (hatch edge 0.5)
+    (priority 3)
     (connect_pads (clearance 0))
     (min_thickness 0.25) (filled_areas_thickness no)
@@
     (polygon
       (pts
-        (xy 238.76 164.465)
-        (xy 251.46 164.465)
-        (xy 251.46 177.8)
-        (xy 238.76 177.8)
+        (xy 75.565 192.405)
+        (xy 63.5 192.405)
+        (xy 63.5 53.34)
+        (xy 75.565 53.34)
       )
     )
   )
-  (zone (net 0) (net_name "") (layer "B.Mask") (hatch edge 0.5)
+  (zone (net 245) (net_name "GND") (layer "B.Cu") (hatch edge 0.5)
+    (priority 2)
     (connect_pads (clearance 0))
     (min_thickness 0.25) (filled_areas_thickness no)
@@
     (polygon
       (pts
-        (xy 69.85 101.6)
-        (xy 63.5 101.6)
-        (xy 63.5 90.17)
-        (xy 69.85 90.17)
+        (xy 251.46 115.57)
+        (xy 251.46 212.09)
+        (xy 121.92 212.09)
+        (xy 121.92 206.375)
+        (xy 236.22 206.375)
+        (xy 236.22 115.57)
       )
     )

Commit message: add cic and wram to board
Parts:
- added U6: WRAM, Package_SO:TSSOP-64_6.1x17mm_P0.5mm, F.Cu at (179.2, 170.9)
- added U7: ~, Package_SO:SSOP-18_4.4x6.5mm_P0.65mm, F.Cu at (223.4, 187.9)
- P1: footprint Connector_DIN:DIN41612_R_2x32_Male_Vertical_THT -> SNES_Library:CASSETTE
- moved R82 13.1 mm to (215.6, 163.2)
- moved C94 3.24 mm to (218.4, 121.9)
- moved C93 3.18 mm to (211.1, 167.6)
- moved DA2 2.34 mm to (229.5, 159.4)
- moved DA3 2.34 mm to (229.5, 163.8)
- moved DA4 2.34 mm to (229.4, 168.2)
- moved DA5 2.34 mm to (229.4, 172.7)
Connections:
- U1 pad 10: unconnected-(U1-A16-Pad10) -> /CA16
- U1 pad 100: unconnected-(U1-A7-Pad100) -> /CA7
- U1 pad 11: unconnected-(U1-A17-Pad11) -> /CA17
- U1 pad 12: unconnected-(U1-A18-Pad12) -> /CA18
- U1 pad 13: unconnected-(U1-A19-Pad13) -> /CA19
- U1 pad 14: unconnected-(U1-A20-Pad14) -> /CA20
- U1 pad 15: unconnected-(U1-A21-Pad15) -> /CA21
- U1 pad 16: unconnected-(U1-A22-Pad16) -> /CA22
- U1 pad 17: unconnected-(U1-A23-Pad17) -> /CA23
- U1 pad 2: unconnected-(U1-A8-Pad2) -> /CA8
- U1 pad 3: unconnected-(U1-A9-Pad3) -> /CA9
- U1 pad 4: unconnected-(U1-A10-Pad4) -> /CA10
- U1 pad 5: unconnected-(U1-A11-Pad5) -> /CA11
- U1 pad 6: unconnected-(U1-A12-Pad6) -> /CA12
- U1 pad 60: unconnected-(U1-D0-Pad60) -> /D0
- U1 pad 61: unconnected-(U1-D1-Pad61) -> /D1
- U1 pad 62: unconnected-(U1-D2-Pad62) -> /D2
- U1 pad 63: unconnected-(U1-D3-Pad63) -> /D3
- U1 pad 64: unconnected-(U1-D4-Pad64) -> /D4
- U1 pad 65: unconnected-(U1-D5-Pad65) -> /D5
- U1 pad 66: unconnected-(U1-D6-Pad66) -> /D6
- U1 pad 67: unconnected-(U1-D7-Pad67) -> /D7
- U1 pad 7: unconnected-(U1-A13-Pad7) -> /CA13
- U1 pad 8: unconnected-(U1-A14-Pad8) -> /CA14
- U1 pad 9: unconnected-(U1-A15-Pad9) -> /CA15
- U1 pad 93: unconnected-(U1-A0-Pad93) -> /CA0
- U1 pad 94: unconnected-(U1-A1-Pad94) -> /CA1
- U1 pad 95: unconnected-(U1-A2-Pad95) -> /CA2
- U1 pad 96: unconnected-(U1-A3-Pad96) -> /CA3
- U1 pad 97: unconnected-(U1-A4-Pad97) -> /CA4
- U1 pad 98: unconnected-(U1-A5-Pad98) -> /CA5
- U1 pad 99: unconnected-(U1-A6-Pad99) -> /CA6
- U2 pad 14: unconnected-(U2-D7-Pad14) -> /D7
- U2 pad 15: unconnected-(U2-D6-Pad15) -> /D6
- U2 pad 16: unconnected-(U2-D5-Pad16) -> /D5
- U2 pad 17: unconnected-(U2-D4-Pad17) -> /D4
- U2 pad 18: unconnected-(U2-D3-Pad18) -> /D3
- U2 pad 19: unconnected-(U2-D2-Pad19) -> /D2
- U2 pad 20: unconnected-(U2-D1-Pad20) -> /D1
- U2 pad 21: unconnected-(U2-D0-Pad21) -> /D0
- U3 pad 10: unconnected-(U3-D5-Pad10) -> /D5
- U3 pad 11: unconnected-(U3-D4-Pad11) -> /D4
- U3 pad 12: unconnected-(U3-D3-Pad12) -> /D3
- U3 pad 13: unconnected-(U3-D2-Pad13) -> /D2
- U3 pad 14: unconnected-(U3-D1-Pad14) -> /D1
- U3 pad 15: unconnected-(U3-D0-Pad15) -> /D0
- U3 pad 8: unconnected-(U3-D7-Pad8) -> /D7
- U3 pad 9: unconnected-(U3-D6-Pad9) -> /D6
Other:
- outline, holes or cut-outs redrawn

Commit message: rename cic
Parts:
- U8: renamed from U7; value ~ -> CIC
- moved P1 9.94 mm to (153.3, 180.1)
- moved U1 2.62 mm to (213.4, 170.8)
- moved U8 1.58 mm to (224.8, 188.6)
- moved U2 0.77 mm to (215.6, 130.3)
Connections:
- U8 pad 18: unconnected-(U7-VCC-Pad18) -> VCC
- U8 pad 9: unconnected-(U7-GND-Pad9) -> GND

Commit message: cartridge port again
Parts:
- moved P1 47.1 mm to (151.0, 133.1)
- moved P3 1.42 mm to (104.1, 202.6)
Routing:
- net Net-(P3-Pin_2): track 20.3 -> 4.17 mm
Other:
- outline, holes or cut-outs redrawn
