File: nonSNES.kicad_pcb (KiCad board)
At the start: 2 copper layers, 188 x 158.8 mm, 55 parts, among them J1 Jack-DC, P1 CASSETTE, P2 Conn_2Rows-11Pins, P3 Conn_01x02_Male, T1 L_Coupled, U1 CPU, U12 L7805, U2 PPU1, U3 PPU2, U4 MS62256CL-10FC, U5 MS62256CL-10FC, U6 WRAM, U8 CIC, X1 Crystal

Commit message: wire cic and reset sw
Parts:
- added C29: 0.1u, Capacitor_SMD:C_0805_2012Metric, B.Cu at (214.3, 185.4)
- added C62: 2.2u, Capacitor_SMD:C_0805_2012Metric, B.Cu at (214.3, 188.4)
- added C85: 0.1u, Capacitor_SMD:C_0805_2012Metric, B.Cu at (214.3, 191.4)
- added SW1: RESET SW, Button_Switch_THT:SW_MEC_5GTH9, F.Cu at (219.1, 89.5)
- moved J1 0.63 mm to (72.4, 198.8)
Connections:
- P1 pad 1: (no net) -> unconnected-(P1-MCK_21M-Pad1)
- P1 pad 10: (no net) -> /CA7
- P1 pad 11: (no net) -> /CA6
- P1 pad 12: (no net) -> /CA5
- P1 pad 13: (no net) -> /CA4
- P1 pad 14: (no net) -> /CA3
- P1 pad 15: (no net) -> /CA2
- P1 pad 16: (no net) -> /CA1
- P1 pad 17: (no net) -> /CA0
- P1 pad 18: (no net) -> unconnected-(P1-IRQ-Pad18)
- P1 pad 19: (no net) -> /D0
- P1 pad 2: (no net) -> unconnected-(P1-EXPAND-Pad2)
- P1 pad 20: (no net) -> /D1
- P1 pad 21: (no net) -> /D2
- P1 pad 22: (no net) -> /D3
- P1 pad 23: (no net) -> unconnected-(P1-RD-Pad23)
- P1 pad 24: (no net) -> unconnected-(P1-CIC0-Pad24)
- P1 pad 25: (no net) -> unconnected-(P1-CIC2-Pad25)
- P1 pad 26: (no net) -> unconnected-(P1-RESET-Pad26)
- P1 pad 27: (no net) -> unconnected-(P1-+5V-Pad27)
- P1 pad 28: (no net) -> unconnected-(P1-PA0-Pad28)
- P1 pad 29: (no net) -> unconnected-(P1-PA2-Pad29)
- P1 pad 3: (no net) -> unconnected-(P1-PA6-Pad3)
- P1 pad 30: (no net) -> unconnected-(P1-PA4-Pad30)
- P1 pad 31: (no net) -> unconnected-(P1-SOUND-L-Pad31)
- P1 pad 32: (no net) -> unconnected-(P1-WRAMSEL-Pad32)
- P1 pad 33: (no net) -> unconnected-(P1-REFRESH-Pad33)
- P1 pad 34: (no net) -> unconnected-(P1-PA7-Pad34)
- P1 pad 35: (no net) -> unconnected-(P1-PAWR-Pad35)
- P1 pad 36: (no net) -> unconnected-(P1-GND-Pad36)
- P1 pad 37: (no net) -> /CA12
- P1 pad 38: (no net) -> /CA13
- P1 pad 39: (no net) -> /CA14
- P1 pad 4: (no net) -> unconnected-(P1-PARD-Pad4)
- P1 pad 40: (no net) -> /CA15
- P1 pad 41: (no net) -> /CA16
- P1 pad 42: (no net) -> /CA17
- P1 pad 43: (no net) -> /CA18
- P1 pad 44: (no net) -> /CA19
- P1 pad 45: (no net) -> /CA20
- P1 pad 46: (no net) -> /CA21
- P1 pad 47: (no net) -> /CA22
- P1 pad 48: (no net) -> /CA23
- P1 pad 49: (no net) -> unconnected-(P1-ROMSEL-Pad49)
- P1 pad 5: (no net) -> unconnected-(P1-GND-Pad5)
- P1 pad 50: (no net) -> /D4
- P1 pad 51: (no net) -> /D5
- P1 pad 52: (no net) -> /D6
- P1 pad 53: (no net) -> /D7
- P1 pad 54: (no net) -> unconnected-(P1-WR-Pad54)
- P1 pad 55: (no net) -> unconnected-(P1-CIC1-Pad55)
- P1 pad 56: (no net) -> unconnected-(P1-CIC3-Pad56)
- P1 pad 57: (no net) -> unconnected-(P1-SYSCK-Pad57)
- P1 pad 58: (no net) -> unconnected-(P1-+5V-Pad58)
- P1 pad 59: (no net) -> unconnected-(P1-PA1-Pad59)
- P1 pad 6: (no net) -> /CA11
- P1 pad 60: (no net) -> unconnected-(P1-PA3-Pad60)
- P1 pad 61: (no net) -> unconnected-(P1-PA5-Pad61)
- P1 pad 62: (no net) -> unconnected-(P1-SOUND-R-Pad62)
- P1 pad 7: (no net) -> /CA10
- P1 pad 8: (no net) -> /CA9
- P1 pad 9: (no net) -> /CA8
- U8 pad 3: unconnected-(U8-P02-Pad3) -> Net-(U8-P02)
- U8 pad 4: unconnected-(U8-P03-Pad4) -> VCC
- U8 pad 8: unconnected-(U8-RES-Pad8) -> Net-(U8-RES)
Routing:
- net Net-(C30-Pad2): track 18.8 -> 0.00 mm
- net Net-(P3-Pin_2): track 4.17 -> 18.8 mm
- net Net-(C30-Pad1): track 16.6 -> 17.8 mm
- net GND: vias 15 -> 24
Other:
- outline, holes or cut-outs redrawn

Commit message: vias, sw
Parts:
- moved SW1 2.01 mm to (221.0, 88.9)
- moved T1 0.99 mm to (83.2, 193.7)
- moved J1 0.87 mm to (71.8, 199.4)
Routing:
- net Net-(C30-Pad1): track 17.8 -> 15.7 mm
- net GND: vias 24 -> 32
Other:
- outline, holes or cut-outs redrawn
Changed lines of the file:
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@@
   )
   (footprint "SNES_Library:DcJack" (layer "F.Cu")
-    (at 72.39 198.755)
+    (at 71.795 199.39)
     (property "Sheetfile" "nonSNES.kicad_sch")
     (property "Sheetname" "")
@@
   )
   (footprint "Button_Switch_THT:SW_MEC_5GTH9" (layer "F.Cu")
-    (at 219.075 89.535 180)
+    (at 220.98 88.9 180)
     (descr "MEC 5G single pole normally-open tactile switch https://cdn.sos.sk/productdata/80/f6/aabf7be6/5gth9358222.pdf")
     (tags "switch normally-open pushbutton push-button")
@@
   )
   (footprint "Inductor_SMD:L_CommonMode_Delevan_4222" (layer "F.Cu")
-    (at 83.82 192.98 90)
+    (at 83.185 193.735 90)
     (descr "API Delevan, Surface Mount Common Mode Bead, 4222 4222R, http://www.delevan.com/seriesPDFs/4222.pdf")
     (tags "surface mount common mode bead")
@@
   (gr_circle (center 108.585 57.785) (end 112.395 57.785)
     (stroke (width 0.15) (type solid)) (fill solid) (layer "B.Mask"))
-  (gr_circle (center 98.425 176.467123) (end 101.6 177.102123)
+  (gr_circle (center 99.757877 175.895) (end 102.932877 176.53)
     (stroke (width 0.15) (type solid)) (fill solid) (layer "B.Mask"))
   (gr_circle (center 125.73 208.915) (end 129.54 208.915)
@@
   (gr_rect (start 88.265 195.58) (end 96.52 212.09)
     (stroke (width 0.15) (type solid)) (fill solid) (layer "F.Mask"))
+  (gr_circle (center 67.945 75.565) (end 70.485 75.565)
+    (stroke (width 0.15) (type solid)) (fill solid) (layer "F.Mask"))
   (gr_poly
     (pts
@@
     )
     (stroke (width 0.15) (type solid)) (fill solid) (layer "F.Mask"))
-  (gr_rect (start 71.755 53.34) (end 128.27 64.77)
+  (gr_rect (start 71.755 53.34) (end 130.175 64.77)
     (stroke (width 0.15) (type solid)) (fill solid) (layer "F.Mask"))
   (gr_rect (start 143.51 53.34) (end 158.75 88.9)
@@
   (gr_line (start 226.06 196.85) (end 236.22 196.85)
     (stroke (width 0.1) (type solid)) (layer "Edge.Cuts"))
-  (gr_circle (center 67.945 75.565) (end 67.945 74.295)
+  (gr_circle (center 67.945 75.565) (end 69.85 75.565)
     (stroke (width 0.1) (type default)) (fill none) (layer "Edge.Cuts"))
   (gr_arc (start 78.105 55.88) (mid 80.01 57.785) (end 78.105 59.69)
@@
   (gr_line (start 63.5 204.47) (end 78.74 204.47)
     (stroke (width 0.1) (type solid)) (layer "Edge.Cuts"))
-  (gr_circle (center 98.425 176.467123) (end 98.425 174.562123)
+  (gr_circle (center 99.695 175.895) (end 99.695 173.99)
     (stroke (width 0.1) (type default)) (fill none) (layer "Edge.Cuts"))
   (gr_line (start 156.21 198.12) (end 156.21 212.09)
@@
   (segment (start 116.586 208.534) (end 116.586 207.127974) (width 1.27) (layer "F.Cu") (net 1))
   (segment (start 116.957974 207.127974) (end 114.3 204.47) (width 1.27) (layer "F.Cu") (net 1))
-  (segment (start 85.09 201.93) (end 85.09 196.73) (width 1.27) (layer "F.Cu") (net 95))
-  (segment (start 74.89 200.62) (end 76.2 201.93) (width 1.27) (layer "F.Cu") (net 95))
-  (segment (start 74.89 198.755) (end 74.89 200.62) (width 1.27) (layer "F.Cu") (net 95))
-  (segment (start 76.2 201.93) (end 85.09 201.93) (width 1.27) (layer "F.Cu") (net 95))
+  (segment (start 74.295 200.025) (end 74.295 199.39) (width 1.27) (layer "F.Cu") (net 95))
+  (segment (start 76.2 201.93) (end 74.295 200.025) (width 1.27) (layer "F.Cu") (net 95))
+  (segment (start 83.82 201.93) (end 84.455 201.295) (width 1.27) (layer "F.Cu") (net 95))
+  (segment (start 84.455 201.295) (end 84.455 197.485) (width 1.27) (layer "F.Cu") (net 95))
+  (segment (start 76.2 201.93) (end 83.82 201.93) (width 1.27) (layer "F.Cu") (net 95))
   (segment (start 232.095 143.51) (end 233.585 142.02) (width 0.25) (layer "B.Cu") (net 244))
   (segment (start 233.585 142.02) (end 238.22 142.02) (width 0.25) (layer "B.Cu") (net 244))
@@
   (segment (start 238.22 142.02) (end 242.16 138.08) (width 0.25) (layer "B.Cu") (net 244))
   (via (at 235.585 138.43) (size 0.8) (drill 0.4) (layers "F.Cu" "B.Cu") (net 245))
+  (via (at 130.175 55.245) (size 0.8) (drill 0.4) (layers "F.Cu" "B.Cu") (free) (net 245))
   (via (at 235.585 123.19) (size 0.8) (drill 0.4) (layers "F.Cu" "B.Cu") (net 245))
   (via (at 95.25 56.515) (size 0.8) (drill 0.4) (layers "F.Cu" "B.Cu") (free) (net 245))
-  (via (at 74.93 71.755) (size 0.8) (drill 0.4) (layers "F.Cu" "B.Cu") (free) (net 245))
+  (via (at 74.295 71.12) (size 0.8) (drill 0.4) (layers "F.Cu" "B.Cu") (free) (net 245))
   (via (at 83.185 62.865) (size 0.8) (drill 0.4) (layers "F.Cu" "B.Cu") (free) (net 245))
   (via (at 235.585 128.27) (size 0.8) (drill 0.4) (layers "F.Cu" "B.Cu") (net 245))
-  (via (at 74.93 67.31) (size 0.8) (drill 0.4) (layers "F.Cu" "B.Cu") (free) (net 245))
+  (via (at 74.295 67.31) (size 0.8) (drill 0.4) (layers "F.Cu" "B.Cu") (free) (net 245))
   (via (at 235.585 125.73) (size 0.8) (drill 0.4) (layers "F.Cu" "B.Cu") (net 245))
-  (via (at 78.74 67.31) (size 0.8) (drill 0.4) (layers "F.Cu" "B.Cu") (free) (net 245))
+  (via (at 78.105 67.31) (size 0.8) (drill 0.4) (layers "F.Cu" "B.Cu") (free) (net 245))
+  (via (at 165.1 66.675) (size 0.8) (drill 0.4) (layers "F.Cu" "B.Cu") (free) (net 245))
   (via (at 67.945 63.5) (size 0.8) (drill 0.4) (layers "F.Cu" "B.Cu") (free) (net 245))
   (via (at 90.805 60.325) (size 0.8) (drill 0.4) (layers "F.Cu" "B.Cu") (free) (net 245))
   (via (at 235.585 143.51) (size 0.8) (drill 0.4) (layers "F.Cu" "B.Cu") (net 245))
   (via (at 235.585 133.35) (size 0.8) (drill 0.4) (layers "F.Cu" "B.Cu") (net 245))
-  (via (at 74.93 75.565) (size 0.8) (drill 0.4) (layers "F.Cu" "B.Cu") (free) (net 245))
+  (via (at 160.02 60.96) (size 0.8) (drill 0.4) (layers "F.Cu" "B.Cu") (free) (net 245))
+  (via (at 165.1 60.96) (size 0.8) (drill 0.4) (layers "F.Cu" "B.Cu") (free) (net 245))
+  (via (at 74.295 74.295) (size 0.8) (drill 0.4) (layers "F.Cu" "B.Cu") (free) (net 245))
   (via (at 90.805 56.515) (size 0.8) (drill 0.4) (layers "F.Cu" "B.Cu") (free) (net 245))
-  (via (at 78.74 62.865) (size 0.8) (drill 0.4) (layers "F.Cu" "B.Cu") (free) (net 245))
+  (via (at 78.105 62.865) (size 0.8) (drill 0.4) (layers "F.Cu" "B.Cu") (free) (net 245))
   (via (at 235.585 130.81) (size 0.8) (drill 0.4) (layers "F.Cu" "B.Cu") (net 245))
   (via (at 86.36 56.515) (size 0.8) (drill 0.4) (layers "F.Cu" "B.Cu") (free) (net 245))
   (via (at 70.485 67.31) (size 0.8) (drill 0.4) (layers "F.Cu" "B.Cu") (free) (net 245))
   (via (at 86.36 60.325) (size 0.8) (drill 0.4) (layers "F.Cu" "B.Cu") (free) (net 245))
+  (via (at 160.02 55.245) (size 0.8) (drill 0.4) (layers "F.Cu" "B.Cu") (free) (net 245))
   (via (at 95.25 60.325) (size 0.8) (drill 0.4) (layers "F.Cu" "B.Cu") (free) (net 245))
+  (via (at 130.175 60.325) (size 0.8) (drill 0.4) (layers "F.Cu" "B.Cu") (free) (net 245))
+  (via (at 160.02 66.675) (size 0.8) (drill 0.4) (layers "F.Cu" "B.Cu") (free) (net 245))
+  (via (at 165.1 55.245) (size 0.8) (drill 0.4) (layers "F.Cu" "B.Cu") (free) (net 245))
   (via (at 235.585 135.89) (size 0.8) (drill 0.4) (layers "F.Cu" "B.Cu") (net 245))
-  (via (at 67.945 69.85) (size 0.8) (drill 0.4) (layers "F.Cu" "B.Cu") (free) (net 245))
+  (via (at 67.945 70.485) (size 0.8) (drill 0.4) (layers "F.Cu" "B.Cu") (free) (net 245))
   (via (at 235.585 140.97) (size 0.8) (drill 0.4) (layers "F.Cu" "B.Cu") (net 245))
   (segment (start 233.995 135.89) (end 235.585 135.89) (width 1) (layer "B.Cu") (net 245))

Commit message: connector
Parts:
- P2: footprint Connector_JST:JST_ZE_B11B-ZESK-D_1x11_P1.50mm_Vertical -> SNES_Library:JST_ZE_Controllers
- moved P2 7.51 mm to (244.2, 132.1)
- moved C37 0.86 mm to (233.0, 137.6)
- moved R85 0.86 mm to (228.9, 137.6)
- moved C41 0.86 mm to (233.0, 127.4)
- moved C42 0.86 mm to (233.0, 124.9)
- moved C43 0.86 mm to (233.0, 122.3)
- moved R89 0.86 mm to (228.9, 127.4)
- moved R90 0.86 mm to (228.9, 124.9)
- moved R91 0.86 mm to (228.9, 122.3)
- moved C35 0.85 mm to (233.0, 142.7)
- moved C36 0.85 mm to (233.0, 140.1)
- moved C38 0.85 mm to (233.0, 135.0)
- moved C39 0.85 mm to (233.0, 132.5)
- moved C40 0.85 mm to (233.0, 130.0)
- moved R83 0.85 mm to (228.9, 142.7)
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Routing:
- net Net-(P2-Pin_5): track 15.3 -> 4.10 mm
- net Net-(P2-Pin_8): track 13.6 -> 3.79 mm
- net Net-(P2-Pin_6): track 12.9 -> 4.10 mm
- net Net-(P2-Pin_7): track 15.3 -> 6.81 mm
- net Net-(P2-Pin_3): track 16.6 -> 8.98 mm
- net Net-(P2-Pin_9): track 16.2 -> 8.91 mm
- net Net-(P2-Pin_10): track 14.4 -> 8.86 mm
- net Net-(P2-Pin_2): track 14.6 -> 9.05 mm
- net Net-(P2-Pin_4): track 13.8 -> 9.11 mm

Commit message: move caps around again
Parts:
- moved C107 14.3 mm to (179.1, 115.6)
- moved C92 7.43 mm to (191.1, 129.5)
- moved C97 1.85 mm to (218.4, 105.4)
- moved P2 1.11 mm to (244.1, 133.2)
- moved C95 0.71 mm to (189.9, 105.1)
- moved C94 0.63 mm to (219.1, 121.9)
Routing:
- net GND: vias 32 -> 35
Other:
- outline, holes or cut-outs redrawn
Changed lines of the file:
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@@
   )
   (footprint "SNES_Library:JST_ZE_Controllers" (layer "F.Cu")
-    (at 244.16 132.07 90)
+    (at 244.13 133.18 90)
     (descr "JST ZE series connector, B11B-ZESK-D (http://www.jst-mfg.com/product/pdf/eng/eZE.pdf), generated with kicad-footprint-generator")
     (tags "connector JST ZE side entry")
@@
     (property "ki_keywords" "R res resistor")
     (attr smd)
-    (fp_text reference "R90" (at 3.81 0) (layer "B.SilkS")
+    (fp_text reference "R90" (at 5.3575 0) (layer "B.SilkS")
         (effects (font (size 1 1) (thickness 0.15)) (justify mirror))
     )
@@
   )
   (footprint "Capacitor_SMD:C_0805_2012Metric" (layer "B.Cu")
-    (at 190.5 105.41 90)
+    (at 189.865 105.09 90)
     (descr "Capacitor SMD 0805 (2012 Metric), square (rectangular) end terminal, IPC_7351 nominal, (Body size source: IPC-SM-782 page 76, https://www.pcb-3d.com/wordpress/wp-content/uploads/ipc-sm-782a_amendment_1_and_2.pdf, https://docs.google.com/spreadsheets/d/1BsfQQcO9C6DZCsRaXUlFlo91Tg2WpOkGARC1WS5S8t0/edit?usp=sharing), generated with kicad-footprint-generator")
     (tags "capacitor")
@@
     (property "ki_keywords" "R res resistor")
     (attr smd)
-    (fp_text reference "R89" (at 3.81 0) (layer "B.SilkS")
+    (fp_text reference "R89" (at 5.3575 0) (layer "B.SilkS")
         (effects (font (size 1 1) (thickness 0.15)) (justify mirror))
     )
@@
   )
   (footprint "Capacitor_SMD:C_0805_2012Metric" (layer "B.Cu")
-    (at 218.44 121.92 180)
+    (at 219.075 121.92 180)
     (descr "Capacitor SMD 0805 (2012 Metric), square (rectangular) end terminal, IPC_7351 nominal, (Body size source: IPC-SM-782 page 76, https://www.pcb-3d.com/wordpress/wp-content/uploads/ipc-sm-782a_amendment_1_and_2.pdf, https://docs.google.com/spreadsheets/d/1BsfQQcO9C6DZCsRaXUlFlo91Tg2WpOkGARC1WS5S8t0/edit?usp=sharing), generated with kicad-footprint-generator")
     (tags "capacitor")
@@
   )
   (footprint "Capacitor_SMD:C_0805_2012Metric" (layer "B.Cu")
-    (at 185.74 128.27 180)
+    (at 179.07 115.57 180)
     (descr "Capacitor SMD 0805 (2012 Metric), square (rectangular) end terminal, IPC_7351 nominal, (Body size source: IPC-SM-782 page 76, https://www.pcb-3d.com/wordpress/wp-content/uploads/ipc-sm-782a_amendment_1_and_2.pdf, https://docs.google.com/spreadsheets/d/1BsfQQcO9C6DZCsRaXUlFlo91Tg2WpOkGARC1WS5S8t0/edit?usp=sharing), generated with kicad-footprint-generator")
     (tags "capacitor")
@@
   )
   (footprint "Capacitor_SMD:C_0805_2012Metric" (layer "B.Cu")
-    (at 188.595 122.555 180)
+    (at 191.135 129.54 180)
     (descr "Capacitor SMD 0805 (2012 Metric), square (rectangular) end terminal, IPC_7351 nominal, (Body size source: IPC-SM-782 page 76, https://www.pcb-3d.com/wordpress/wp-content/uploads/ipc-sm-782a_amendment_1_and_2.pdf, https://docs.google.com/spreadsheets/d/1BsfQQcO9C6DZCsRaXUlFlo91Tg2WpOkGARC1WS5S8t0/edit?usp=sharing), generated with kicad-footprint-generator")
     (tags "capacitor")
@@
   )
   (footprint "Capacitor_SMD:C_0805_2012Metric" (layer "B.Cu")
-    (at 216.662 104.902 -90)
+    (at 218.44 105.41 -90)
     (descr "Capacitor SMD 0805 (2012 Metric), square (rectangular) end terminal, IPC_7351 nominal, (Body size source: IPC-SM-782 page 76, https://www.pcb-3d.com/wordpress/wp-content/uploads/ipc-sm-782a_amendment_1_and_2.pdf, https://docs.google.com/spreadsheets/d/1BsfQQcO9C6DZCsRaXUlFlo91Tg2WpOkGARC1WS5S8t0/edit?usp=sharing), generated with kicad-footprint-generator")
     (tags "capacitor")
@@
     )
   )
+  (gr_rect (start 247.65 62.23) (end 251.46 66.04)
+    (stroke (width 0.15) (type solid)) (fill solid) (layer "B.Paste"))
+  (gr_rect (start 247.65 98.425) (end 251.46 102.235)
+    (stroke (width 0.15) (type solid)) (fill solid) (layer "B.Paste"))
   (gr_circle (center 73.025 159.447877) (end 76.2 160.082877)
     (stroke (width 0.15) (type solid)) (fill solid) (layer "B.Mask"))
@@
   (gr_rect (start 143.51 53.34) (end 158.75 88.9)
     (stroke (width 0.15) (type solid)) (fill solid) (layer "F.Mask"))
-  (gr_circle (center 241.935 82.55) (end 241.935 81.28)
+  (gr_circle (center 242.57 83.185) (end 242.57 81.915)
     (stroke (width 0.1) (type default)) (fill none) (layer "Edge.Cuts"))
   (gr_line (start 126.365 58.42) (end 126.365 53.34)
@@
   (gr_circle (center 73.025 159.385) (end 73.025 157.48)
     (stroke (width 0.1) (type default)) (fill none) (layer "Edge.Cuts"))
-  (gr_circle (center 247.015 208.28) (end 247.015 207.01)
-    (stroke (width 0.1) (type default)) (fill none) (layer "Edge.Cuts"))
+  (gr_line (start 245.745 208.28) (end 245.745 207.01)
+    (stroke (width 0.1) (type default)) (layer "Edge.Cuts"))
   (gr_line (start 168.275 53.34) (end 168.275 68.58)
     (stroke (width 0.1) (type solid)) (layer "Edge.Cuts"))
@@
   (gr_circle (center 70.485 150.495) (end 70.485 149.225)
     (stroke (width 0.1) (type default)) (fill none) (layer "Edge.Cuts"))
-  (gr_circle (center 241.935 88.265) (end 241.935 88.9)
+  (gr_circle (center 242.57 88.9) (end 242.57 89.535)
     (stroke (width 0.1) (type default)) (fill none) (layer "Edge.Cuts"))
   (gr_line (start 251.46 212.09) (end 251.46 53.34)
@@
   (gr_circle (center 212.09 200.025) (end 212.09 198.12)
     (stroke (width 0.1) (type default)) (fill none) (layer "Edge.Cuts"))
+  (gr_arc (start 248.285 208.28) (mid 247.015 209.55) (end 245.745 208.28)
+    (stroke (width 0.1) (type default)) (layer "Edge.Cuts"))
   (gr_line (start 201.93 212.09) (end 226.06 212.09)
     (stroke (width 0.1) (type solid)) (layer "Edge.Cuts"))
@@
   (gr_line (start 63.5 204.47) (end 78.74 204.47)
     (stroke (width 0.1) (type solid)) (layer "Edge.Cuts"))
+  (gr_line (start 248.285 207.01) (end 248.285 208.28)
+    (stroke (width 0.1) (type default)) (layer "Edge.Cuts"))
+  (gr_arc (start 245.745 207.01) (mid 247.015 205.74) (end 248.285 207.01)
+    (stroke (width 0.1) (type default)) (layer "Edge.Cuts"))
   (gr_circle (center 99.695 175.895) (end 99.695 173.99)
     (stroke (width 0.1) (type default)) (fill none) (layer "Edge.Cuts"))
@@
   (via (at 235.585 137.575) (size 0.8) (drill 0.4) (layers "F.Cu" "B.Cu") (net 245))
   (via (at 130.175 55.245) (size 0.8) (drill 0.4) (layers "F.Cu" "B.Cu") (free) (net 245))
+  (via (at 241.3 57.15) (size 0.8) (drill 0.4) (layers "F.Cu" "B.Cu") (free) (net 245))
   (via (at 235.585 122.335) (size 0.8) (drill 0.4) (layers "F.Cu" "B.Cu") (net 245))
   (via (at 95.25 56.515) (size 0.8) (drill 0.4) (layers "F.Cu" "B.Cu") (free) (net 245))
   (via (at 74.295 71.12) (size 0.8) (drill 0.4) (layers "F.Cu" "B.Cu") (free) (net 245))
+  (via (at 234.95 57.15) (size 0.8) (drill 0.4) (layers "F.Cu" "B.Cu") (free) (net 245))
+  (via (at 228.6 57.15) (size 0.8) (drill 0.4) (layers "F.Cu" "B.Cu") (free) (net 245))
   (via (at 83.185 62.865) (size 0.8) (drill 0.4) (layers "F.Cu" "B.Cu") (free) (net 245))
   (via (at 235.585 127.415) (size 0.8) (drill 0.4) (layers "F.Cu" "B.Cu") (net 245))

Commit message: pad and cap
Parts:
- added C67: 1000u, Capacitor_THT:CP_Radial_D16.0mm_P7.50mm, F.Cu at (114.0, 176.5)
- moved C85 13.7 mm to (228.0, 190.5), turned to 90 degrees
- moved C29 11.7 mm to (225.4, 188.9), turned to -90 degrees
- moved C30 2.13 mm to (82.9, 192.4)
- moved C31 2.13 mm to (82.9, 189.2)
- moved DA2 1.43 mm to (231.0, 159.4)
- moved DA3 1.43 mm to (231.0, 163.8)
- moved DA4 1.43 mm to (230.8, 168.2)
- moved DA5 1.43 mm to (230.8, 172.7)
Routing:
- net Net-(C30-Pad2): track 0.00 -> 21.4 mm
