File: nonSNES.kicad_pcb (KiCad board)
At the start: 2 copper layers, 188 x 158.8 mm, 60 parts, among them J1 Jack-DC, P1 CASSETTE, P2 Conn_2Rows-11Pins, P3 Conn_01x02_Male, SW1 RESET SW, T1 L_Coupled, U1 CPU, U12 L7805, U2 PPU1, U3 PPU2, U4 MS62256CL-10FC, U5 MS62256CL-10FC, U6 WRAM, U8 CIC, X1 Crystal

Commit message: vias
Parts:
- moved C67 2.58 mm to (114.4, 179.1)
Routing:
- net GND: vias 35 -> 53
Other:
- outline, holes or cut-outs redrawn
Changed lines of the file:
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@@
   )
   (footprint "Capacitor_THT:CP_Radial_D16.0mm_P7.50mm" (layer "F.Cu")
-    (at 113.962246 176.53)
+    (at 114.42 179.07)
     (descr "CP, Radial series, Radial, pin pitch=7.50mm, , diameter=16mm, Electrolytic Capacitor")
     (tags "CP Radial series Radial pin pitch 7.50mm  diameter 16mm Electrolytic Capacitor")
@@
   (gr_circle (center 92.075 209.55) (end 95.25 209.55)
     (stroke (width 0.15) (type solid)) (fill solid) (layer "B.Mask"))
-  (gr_circle (center 108.585 57.785) (end 112.395 57.785)
+  (gr_circle (center 111.125 57.785) (end 114.935 57.785)
     (stroke (width 0.15) (type solid)) (fill solid) (layer "B.Mask"))
   (gr_circle (center 99.757877 175.895) (end 102.932877 176.53)
@@
   (gr_line (start 145.415 53.34) (end 145.415 66.04)
     (stroke (width 0.1) (type solid)) (layer "Edge.Cuts"))
-  (gr_circle (center 108.585 57.785) (end 108.585 55.88)
+  (gr_circle (center 111.125 57.785) (end 111.125 55.88)
     (stroke (width 0.1) (type default)) (fill none) (layer "Edge.Cuts"))
   (gr_circle (center 241.935 182.88) (end 241.935 181.61)
     (stroke (width 0.1) (type default)) (fill none) (layer "Edge.Cuts"))
-  (gr_circle (center 137.795 198.12) (end 137.795 196.85)
+  (gr_circle (center 137.16 198.755) (end 137.16 197.485)
     (stroke (width 0.1) (type default)) (fill none) (layer "Edge.Cuts"))
   (gr_circle (center 136.525 67.31) (end 136.525 66.04)
@@
   (gr_circle (center 73.025 190.5) (end 73.025 187.96)
     (stroke (width 0.1) (type default)) (fill none) (layer "Edge.Cuts"))
-  (gr_circle (center 137.795 208.28) (end 137.795 207.01)
+  (gr_circle (center 137.16 208.915) (end 137.16 207.645)
     (stroke (width 0.1) (type default)) (fill none) (layer "Edge.Cuts"))
   (gr_line (start 104.14 212.09) (end 78.74 212.09)
@@
   (segment (start 83.82 201.93) (end 84.455 201.295) (width 1.27) (layer "F.Cu") (net 95))
   (segment (start 84.455 201.295) (end 84.455 197.485) (width 1.27) (layer "F.Cu") (net 95))
-  (segment (start 76.2 201.93) (end 83.82 201.93) (width 1.27) (layer "F.Cu") (net 95))
+  (segment (start 76.2 201.93) (end 83.82 201.93) (width 2.54) (layer "F.Cu") (net 95))
   (segment (start 80.645 199.39) (end 76.2 194.945) (width 1.27) (layer "F.Cu") (net 96))
   (segment (start 76.2 194.945) (end 69.215 194.945) (width 1.27) (layer "F.Cu") (net 96))
@@
   (segment (start 233.585 141.165) (end 238.22 141.165) (width 0.25) (layer "B.Cu") (net 244))
   (segment (start 232.095 142.655) (end 229.79 142.655) (width 0.25) (layer "B.Cu") (net 244))
+  (via (at 150.495 69.85) (size 0.8) (drill 0.4) (layers "F.Cu" "B.Cu") (free) (net 245))
+  (via (at 134.62 55.245) (size 0.8) (drill 0.4) (layers "F.Cu" "B.Cu") (free) (net 245))
   (via (at 235.585 137.575) (size 0.8) (drill 0.4) (layers "F.Cu" "B.Cu") (net 245))
+  (via (at 134.62 60.96) (size 0.8) (drill 0.4) (layers "F.Cu" "B.Cu") (free) (net 245))
   (via (at 130.175 55.245) (size 0.8) (drill 0.4) (layers "F.Cu" "B.Cu") (free) (net 245))
   (via (at 241.3 57.15) (size 0.8) (drill 0.4) (layers "F.Cu" "B.Cu") (free) (net 245))
   (via (at 235.585 122.335) (size 0.8) (drill 0.4) (layers "F.Cu" "B.Cu") (net 245))
+  (via (at 89.535 199.39) (size 0.8) (drill 0.4) (layers "F.Cu" "B.Cu") (free) (net 245))
   (via (at 95.25 56.515) (size 0.8) (drill 0.4) (layers "F.Cu" "B.Cu") (free) (net 245))
-  (via (at 74.295 71.12) (size 0.8) (drill 0.4) (layers "F.Cu" "B.Cu") (free) (net 245))
+  (via (at 74.295 70.485) (size 0.8) (drill 0.4) (layers "F.Cu" "B.Cu") (free) (net 245))
   (via (at 234.95 57.15) (size 0.8) (drill 0.4) (layers "F.Cu" "B.Cu") (free) (net 245))
+  (via (at 143.51 55.245) (size 0.8) (drill 0.4) (layers "F.Cu" "B.Cu") (free) (net 245))
   (via (at 228.6 57.15) (size 0.8) (drill 0.4) (layers "F.Cu" "B.Cu") (free) (net 245))
   (via (at 83.185 62.865) (size 0.8) (drill 0.4) (layers "F.Cu" "B.Cu") (free) (net 245))
   (via (at 235.585 127.415) (size 0.8) (drill 0.4) (layers "F.Cu" "B.Cu") (net 245))
+  (via (at 138.43 60.96) (size 0.8) (drill 0.4) (layers "F.Cu" "B.Cu") (free) (net 245))
   (via (at 74.295 67.31) (size 0.8) (drill 0.4) (layers "F.Cu" "B.Cu") (free) (net 245))
+  (via (at 104.775 197.485) (size 0.8) (drill 0.4) (layers "F.Cu" "B.Cu") (free) (net 245))
   (via (at 235.585 124.875) (size 0.8) (drill 0.4) (layers "F.Cu" "B.Cu") (net 245))
+  (via (at 143.51 60.96) (size 0.8) (drill 0.4) (layers "F.Cu" "B.Cu") (free) (net 245))
   (via (at 78.105 67.31) (size 0.8) (drill 0.4) (layers "F.Cu" "B.Cu") (free) (net 245))
-  (via (at 165.1 66.675) (size 0.8) (drill 0.4) (layers "F.Cu" "B.Cu") (free) (net 245))
+  (via (at 165.1 67.31) (size 0.8) (drill 0.4) (layers "F.Cu" "B.Cu") (free) (net 245))
+  (via (at 89.535 201.93) (size 0.8) (drill 0.4) (layers "F.Cu" "B.Cu") (free) (net 245))
   (via (at 67.945 63.5) (size 0.8) (drill 0.4) (layers "F.Cu" "B.Cu") (free) (net 245))
   (via (at 90.805 60.325) (size 0.8) (drill 0.4) (layers "F.Cu" "B.Cu") (free) (net 245))
   (via (at 235.585 142.655) (size 0.8) (drill 0.4) (layers "F.Cu" "B.Cu") (net 245))
+  (via (at 92.075 196.85) (size 0.8) (drill 0.4) (layers "F.Cu" "B.Cu") (free) (net 245))
+  (via (at 92.075 201.93) (size 0.8) (drill 0.4) (layers "F.Cu" "B.Cu") (free) (net 245))
   (via (at 235.585 132.495) (size 0.8) (drill 0.4) (layers "F.Cu" "B.Cu") (net 245))
-  (via (at 160.02 60.96) (size 0.8) (drill 0.4) (layers "F.Cu" "B.Cu") (free) (net 245))
+  (via (at 89.535 196.85) (size 0.8) (drill 0.4) (layers "F.Cu" "B.Cu") (free) (net 245))
+  (via (at 159.385 60.96) (size 0.8) (drill 0.4) (layers "F.Cu" "B.Cu") (free) (net 245))
+  (via (at 99.695 197.485) (size 0.8) (drill 0.4) (layers "F.Cu" "B.Cu") (free) (net 245))
   (via (at 165.1 60.96) (size 0.8) (drill 0.4) (layers "F.Cu" "B.Cu") (free) (net 245))
+  (via (at 143.51 66.675) (size 0.8) (drill 0.4) (layers "F.Cu" "B.Cu") (free) (net 245))
   (via (at 74.295 74.295) (size 0.8) (drill 0.4) (layers "F.Cu" "B.Cu") (free) (net 245))
   (via (at 90.805 56.515) (size 0.8) (drill 0.4) (layers "F.Cu" "B.Cu") (free) (net 245))
   (via (at 78.105 62.865) (size 0.8) (drill 0.4) (layers "F.Cu" "B.Cu") (free) (net 245))
   (via (at 235.585 129.955) (size 0.8) (drill 0.4) (layers "F.Cu" "B.Cu") (net 245))
+  (via (at 143.51 69.85) (size 0.8) (drill 0.4) (layers "F.Cu" "B.Cu") (free) (net 245))
   (via (at 86.36 56.515) (size 0.8) (drill 0.4) (layers "F.Cu" "B.Cu") (free) (net 245))
   (via (at 70.485 67.31) (size 0.8) (drill 0.4) (layers "F.Cu" "B.Cu") (free) (net 245))
   (via (at 86.36 60.325) (size 0.8) (drill 0.4) (layers "F.Cu" "B.Cu") (free) (net 245))
-  (via (at 160.02 55.245) (size 0.8) (drill 0.4) (layers "F.Cu" "B.Cu") (free) (net 245))
+  (via (at 107.315 197.485) (size 0.8) (drill 0.4) (layers "F.Cu" "B.Cu") (free) (net 245))
+  (via (at 159.385 55.245) (size 0.8) (drill 0.4) (layers "F.Cu" "B.Cu") (free) (net 245))
   (via (at 95.25 60.325) (size 0.8) (drill 0.4) (layers "F.Cu" "B.Cu") (free) (net 245))
-  (via (at 130.175 60.325) (size 0.8) (drill 0.4) (layers "F.Cu" "B.Cu") (free) (net 245))
-  (via (at 160.02 66.675) (size 0.8) (drill 0.4) (layers "F.Cu" "B.Cu") (free) (net 245))
+  (via (at 102.235 197.485) (size 0.8) (drill 0.4) (layers "F.Cu" "B.Cu") (free) (net 245))
+  (via (at 138.43 55.245) (size 0.8) (drill 0.4) (layers "F.Cu" "B.Cu") (free) (net 245))
+  (via (at 130.175 60.96) (size 0.8) (drill 0.4) (layers "F.Cu" "B.Cu") (free) (net 245))
+  (via (at 159.385 67.31) (size 0.8) (drill 0.4) (layers "F.Cu" "B.Cu") (free) (net 245))
   (via (at 165.1 55.245) (size 0.8) (drill 0.4) (layers "F.Cu" "B.Cu") (free) (net 245))
   (via (at 235.585 135.035) (size 0.8) (drill 0.4) (layers "F.Cu" "B.Cu") (net 245))
@@
         (xy 79.375 211.455)
         (xy 96.52 211.455)
-        (xy 96.52 198.12)
-        (xy 111.125 198.12)
-        (xy 96.52 194.31)
-        (xy 88.265 194.31)
+        (xy 96.52 199.39)
+        (xy 112.395 199.39)
+        (xy 96.52 193.675)
+        (xy 88.265 193.675)
         (xy 88.265 204.47)
         (xy 79.375 204.47)

Commit message: copper fill and vias
Routing:
- net GND: vias 53 -> 58
Changed lines of the file:
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@@
   (segment (start 116.957974 207.127974) (end 114.3 204.47) (width 1.27) (layer "F.Cu") (net 1))
   (segment (start 74.295 200.025) (end 74.295 199.39) (width 1.27) (layer "F.Cu") (net 95))
-  (segment (start 76.2 201.93) (end 74.295 200.025) (width 1.27) (layer "F.Cu") (net 95))
-  (segment (start 83.82 201.93) (end 84.455 201.295) (width 1.27) (layer "F.Cu") (net 95))
+  (segment (start 76.2 201.93) (end 74.295 200.025) (width 2.54) (layer "F.Cu") (net 95))
   (segment (start 84.455 201.295) (end 84.455 197.485) (width 1.27) (layer "F.Cu") (net 95))
   (segment (start 76.2 201.93) (end 83.82 201.93) (width 2.54) (layer "F.Cu") (net 95))
+  (segment (start 83.82 201.93) (end 84.455 201.295) (width 1.27) (layer "F.Cu") (net 95))
   (segment (start 80.645 199.39) (end 76.2 194.945) (width 1.27) (layer "F.Cu") (net 96))
   (segment (start 76.2 194.945) (end 69.215 194.945) (width 1.27) (layer "F.Cu") (net 96))
@@
   (via (at 95.25 56.515) (size 0.8) (drill 0.4) (layers "F.Cu" "B.Cu") (free) (net 245))
   (via (at 74.295 70.485) (size 0.8) (drill 0.4) (layers "F.Cu" "B.Cu") (free) (net 245))
+  (via (at 71.12 176.53) (size 0.8) (drill 0.4) (layers "F.Cu" "B.Cu") (free) (net 245))
   (via (at 234.95 57.15) (size 0.8) (drill 0.4) (layers "F.Cu" "B.Cu") (free) (net 245))
   (via (at 143.51 55.245) (size 0.8) (drill 0.4) (layers "F.Cu" "B.Cu") (free) (net 245))
   (via (at 228.6 57.15) (size 0.8) (drill 0.4) (layers "F.Cu" "B.Cu") (free) (net 245))
   (via (at 83.185 62.865) (size 0.8) (drill 0.4) (layers "F.Cu" "B.Cu") (free) (net 245))
+  (via (at 76.2 176.53) (size 0.8) (drill 0.4) (layers "F.Cu" "B.Cu") (free) (net 245))
   (via (at 235.585 127.415) (size 0.8) (drill 0.4) (layers "F.Cu" "B.Cu") (net 245))
+  (via (at 80.645 171.45) (size 0.8) (drill 0.4) (layers "F.Cu" "B.Cu") (free) (net 245))
   (via (at 138.43 60.96) (size 0.8) (drill 0.4) (layers "F.Cu" "B.Cu") (free) (net 245))
   (via (at 74.295 67.31) (size 0.8) (drill 0.4) (layers "F.Cu" "B.Cu") (free) (net 245))
@@
   (via (at 78.105 67.31) (size 0.8) (drill 0.4) (layers "F.Cu" "B.Cu") (free) (net 245))
   (via (at 165.1 67.31) (size 0.8) (drill 0.4) (layers "F.Cu" "B.Cu") (free) (net 245))
-  (via (at 89.535 201.93) (size 0.8) (drill 0.4) (layers "F.Cu" "B.Cu") (free) (net 245))
+  (via (at 89.535 203.2) (size 0.8) (drill 0.4) (layers "F.Cu" "B.Cu") (free) (net 245))
   (via (at 67.945 63.5) (size 0.8) (drill 0.4) (layers "F.Cu" "B.Cu") (free) (net 245))
   (via (at 90.805 60.325) (size 0.8) (drill 0.4) (layers "F.Cu" "B.Cu") (free) (net 245))
   (via (at 235.585 142.655) (size 0.8) (drill 0.4) (layers "F.Cu" "B.Cu") (net 245))
   (via (at 92.075 196.85) (size 0.8) (drill 0.4) (layers "F.Cu" "B.Cu") (free) (net 245))
-  (via (at 92.075 201.93) (size 0.8) (drill 0.4) (layers "F.Cu" "B.Cu") (free) (net 245))
+  (via (at 92.075 203.2) (size 0.8) (drill 0.4) (layers "F.Cu" "B.Cu") (free) (net 245))
   (via (at 235.585 132.495) (size 0.8) (drill 0.4) (layers "F.Cu" "B.Cu") (net 245))
   (via (at 89.535 196.85) (size 0.8) (drill 0.4) (layers "F.Cu" "B.Cu") (free) (net 245))
@@
   (via (at 70.485 67.31) (size 0.8) (drill 0.4) (layers "F.Cu" "B.Cu") (free) (net 245))
   (via (at 86.36 60.325) (size 0.8) (drill 0.4) (layers "F.Cu" "B.Cu") (free) (net 245))
+  (via (at 76.2 171.45) (size 0.8) (drill 0.4) (layers "F.Cu" "B.Cu") (free) (net 245))
   (via (at 107.315 197.485) (size 0.8) (drill 0.4) (layers "F.Cu" "B.Cu") (free) (net 245))
   (via (at 159.385 55.245) (size 0.8) (drill 0.4) (layers "F.Cu" "B.Cu") (free) (net 245))
@@
   (via (at 102.235 197.485) (size 0.8) (drill 0.4) (layers "F.Cu" "B.Cu") (free) (net 245))
   (via (at 138.43 55.245) (size 0.8) (drill 0.4) (layers "F.Cu" "B.Cu") (free) (net 245))
+  (via (at 83.82 177.165) (size 0.8) (drill 0.4) (layers "F.Cu" "B.Cu") (free) (net 245))
   (via (at 130.175 60.96) (size 0.8) (drill 0.4) (layers "F.Cu" "B.Cu") (free) (net 245))
   (via (at 159.385 67.31) (size 0.8) (drill 0.4) (layers "F.Cu" "B.Cu") (free) (net 245))
@@
         (xy 79.375 211.455)
         (xy 96.52 211.455)
-        (xy 96.52 199.39)
-        (xy 112.395 199.39)
-        (xy 96.52 193.675)
+        (xy 96.52 200.025)
+        (xy 112.395 200.025)
+        (xy 112.395 193.675)
+        (xy 93.345 193.675)
+        (xy 93.345 182.245)
+        (xy 88.265 182.245)
         (xy 88.265 193.675)
         (xy 88.265 204.47)
@@
         (xy 130.81 64.77)
         (xy 83.82 64.77)
-        (xy 83.82 71.12)
-        (xy 83.82 181.61)
-        (xy 73.66 181.61)
-        (xy 73.66 189.23)
-        (xy 64.135 189.23)
+        (xy 88.9 71.12)
+        (xy 88.9 181.61)
+        (xy 76.2 181.61)
+        (xy 76.2 192.405)
+        (xy 64.135 192.405)
         (xy 64.135 64.77)
         (xy 64.135 53.975)
@@
     (polygon
       (pts
-        (xy 75.565 192.405)
-        (xy 63.5 192.405)
-        (xy 63.5 53.34)
-        (xy 75.565 53.34)
+        (xy 76.2 192.405)
+        (xy 64.135 192.405)
+        (xy 64.135 53.975)
+        (xy 76.2 53.975)
       )
     )

Commit message: bottom ground
Parts:
- moved C35 0.64 mm to (233.7, 142.7)
- moved C36 0.64 mm to (233.7, 140.1)
- moved C37 0.64 mm to (233.7, 137.6)
- moved C38 0.64 mm to (233.7, 135.0)
- moved C39 0.64 mm to (233.7, 132.5)
- moved C40 0.64 mm to (233.7, 130.0)
- moved C41 0.64 mm to (233.7, 127.4)
- moved C42 0.64 mm to (233.7, 124.9)
- moved C43 0.64 mm to (233.7, 122.3)
- moved C67 0.63 mm to (114.4, 178.4)
Routing:
- net VCC: track 0.00 -> 12.8 mm, vias 0 -> 1
- net Net-(P2-Pin_3): track 8.98 -> 15.3 mm
- net Net-(P2-Pin_2): track 9.05 -> 13.8 mm
- net Net-(P2-Pin_4): track 9.11 -> 12.6 mm
- net Net-(P2-Pin_7): track 6.81 -> 7.44 mm
- net Net-(P2-Pin_8): track 3.79 -> 4.42 mm
- net Net-(P2-Pin_9): track 8.91 -> 9.55 mm
- net Net-(P2-Pin_6): track 4.10 -> 4.74 mm
- net Net-(P2-Pin_5): track 4.10 -> 4.74 mm
- net Net-(P2-Pin_10): track 8.86 -> 9.50 mm
