File: SNSP-CPU-1CHIP/SNSP-CPU-1CHIP.kicad_pcb (KiCad board)
At the start: 2 copper layers, 155.5 x 161.9 mm, 241 parts, among them J1 Jack-DC, P1 CASSETTE, P2 JST 11FE-BT-VK-N, P3 PWR_SW, P4 AVOUT, P5 EXPANSION, Q1 C2412, Q2 C2412, Q3 C2412, SW1 RESET, T1 TDK zjys-2, U1 S-CPUN(5A122), U10 S-MIX, U11 T5290, U2 S-APU, U3 WRAM, U4 32Kx8_SRAM, U5 32Kx8_SRAM, U6 UPD6379A, U7 S-RGB, U8 CIC, U9 L7805, X1 17.734476MHz, X2 24.57MHz

Commit message: remove images
Routing:
- net /~{VBWR}: track 37.2 -> 35.9 mm
- net /~{VAWR}: track 26.3 -> 25.2 mm
