File: SNSP-CPU-1CHIP/SNSP-CPU-1CHIP.kicad_sch (KiCad schematic)
At the start: 237 parts, among them J1 Jack-DC, P1 CASSETTE, P2 FRONT_PANEL_CONNECTOR, P3 PWR_SW, P4 AVOUT, P5 EXPANSION, Q1 C2412, Q2 C2412, Q3 C2412, SW1 RESET, T1 TDK zjys-2, U1 S-CPUN(5A122), U10 S-MIX, U11 Reset Monitor, U2 S-APU, U3 WRAM, U4 32Kx8_SRAM, U5 32Kx8_SRAM, U6 UPD6379A, U7 S-RGB, U8 CIC, U9 L7805, X1 17.734476MHz, X2 24.57MHz

Commit message: finish components
Parts:
- removed C73, C76: ?, Capacitor_SMD:C_0805_2012Metric_Pad1.18x1.45mm_HandSolder, symbol Device:C_Small
- removed H4, H9: MountingHole, MountingHole:MountingHole_3.7mm, symbol Mechanical:MountingHole
- added C55: ?, Capacitor_SMD:C_0805_2012Metric_Pad1.18x1.45mm_HandSolder, symbol Device:C_Small
- added H4, H9: MountingHole, MountingHole:MountingHole_3.7mm_Pad, symbol Mechanical:MountingHole_Pad
- added R31, R5, R6, R7, R8: ?, Resistor_SMD:R_0805_2012Metric_Pad1.20x1.40mm_HandSolder, symbol Device:R_Small
- C78: renamed from C55; value ? -> OS-CON; footprint Capacitor_THT:C_Disc_D4.3mm_W1.9mm_P5.00mm -> Capacitor_THT:CP_Radial_Tantal_D4.5mm_P5.00mm; symbol Device:C_Small -> Device:C_Polarized
- H8: footprint MountingHole:MountingHole_3.7mm -> MountingHole:MountingHole_3.7mm_Pad; symbol Mechanical:MountingHole -> Mechanical:MountingHole_Pad
- P2: value FRONT_PANEL_CONNECTOR -> JST 11FE-BT-VK-N
- TC1: renamed from C20; footprint Capacitor_THT:C_Disc_D4.3mm_W1.9mm_P5.00mm -> Capacitor_THT:CP_Radial_Tantal_D4.5mm_P5.00mm; symbol Device:C_Small -> Device:C_Polarized
- U11: value Reset Monitor -> T5290
- renumbered C75 to C20, C77 to C73
Connections:
- net B: now also R8.2
- net G: now also R7.2
- net GND: now also H8.1, C55.2, H4.1, H9.1, R31.2, R5.2, R6.1, R7.1, R8.1
- net R: now also R6.2
- net at C53.2, R4.1: now also R5.1
- net at C10.1, P1.1 (MCK_21M), R30.2: now also R31.1
- net at U2.26 (XTAL0), X2.3: now also C55.1
Other:
- moved on the sheet: C6, C7, C8

Commit message: remove images
Parts:
- D2, D3, D4, D5: symbol PAL-snes-1chip-schematic-rescue:D_Small_ALT-Device -> Device:D_Small
- RF1: symbol SNES_parts:RF_MODULATOR -> SNES_Library:RFMODULATOR
Other:
- moved on the sheet: D1
Changed lines of the file:
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@@
 	)
 	(junction
-		(at 589.915 25.4)
+		(at 590.55 25.4)
 		(diameter 0)
 		(color 0 0 0 0)
@@
 	)
 	(no_connect
-		(at 582.295 35.56)
+		(at 582.93 35.56)
 	)
 	(no_connect
@@
 	(wire
 		(pts
-			(xy 589.915 25.4) (xy 589.915 30.48)
+			(xy 590.55 25.4) (xy 590.55 30.48)
 		)
 		(stroke
@@
 	(wire
 		(pts
-			(xy 597.535 35.56) (xy 610.87 35.56)
+			(xy 598.17 35.56) (xy 610.87 35.56)
 		)
 		(stroke
@@
 	(wire
 		(pts
-			(xy 381 25.4) (xy 589.915 25.4)
+			(xy 381 25.4) (xy 590.55 25.4)
 		)
 		(stroke
@@
 	(wire
 		(pts
-			(xy 589.915 25.4) (xy 596.9 25.4)
+			(xy 590.55 25.4) (xy 596.9 25.4)
 		)
 		(stroke
@@
 	)
 	(symbol
-		(lib_id "PAL-snes-1chip-schematic-rescue:D_Small_ALT-Device")
+		(lib_id "Device:D_Small")
 		(at 731.52 83.82 0)
 		(unit 1)
@@
 			)
 		)
-		(property "Description" ""
+		(property "Description" "Diode, small symbol"
+			(at 731.52 83.82 0)
+			(hide yes)
+			(show_name no)
+			(do_not_autoplace no)
+			(effects
+				(font
+					(size 1.27 1.27)
+				)
+			)
+		)
+		(property "Sim.Device" "D"
+			(at 731.52 83.82 0)
+			(hide yes)
+			(show_name no)
+			(do_not_autoplace no)
+			(effects
+				(font
+					(size 1.27 1.27)
+				)
+			)
+		)
+		(property "Sim.Pins" "1=K 2=A"
 			(at 731.52 83.82 0)
+			(hide yes)
 			(show_name no)
 			(do_not_autoplace no)
@@
 	)
 	(symbol
-		(lib_id "PAL-snes-1chip-schematic-rescue:D_Small_ALT-Device")
+		(lib_id "Device:D_Small")
 		(at 721.36 83.82 0)
 		(unit 1)
@@
 			)
 		)
-		(property "Description" ""
+		(property "Description" "Diode, small symbol"
 			(at 721.36 83.82 0)
+			(hide yes)
+			(show_name no)
+			(do_not_autoplace no)
+			(effects
+				(font
+					(size 1.27 1.27)
+				)
+			)
+		)
+		(property "Sim.Device" "D"
+			(at 721.36 83.82 0)
+			(hide yes)
+			(show_name no)
+			(do_not_autoplace no)
+			(effects
+				(font
+					(size 1.27 1.27)
+				)
+			)
+		)
+		(property "Sim.Pins" "1=K 2=A"
+			(at 721.36 83.82 0)
+			(hide yes)
 			(show_name no)
 			(do_not_autoplace no)
@@
 	)
 	(symbol
-		(lib_id "PAL-snes-1chip-schematic-rescue:D_Small_ALT-Device")
+		(lib_id "Device:D_Small")
 		(at 731.52 92.71 0)
 		(unit 1)
@@
 			)
 		)
-		(property "Description" ""
+		(property "Description" "Diode, small symbol"
 			(at 731.52 92.71 0)
+			(hide yes)
+			(show_name no)
+			(do_not_autoplace no)
+			(effects
+				(font
+					(size 1.27 1.27)
+				)
+			)
+		)
+		(property "Sim.Device" "D"
+			(at 731.52 92.71 0)
+			(hide yes)
+			(show_name no)
+			(do_not_autoplace no)
+			(effects
+				(font
+					(size 1.27 1.27)
+				)
+			)
+		)
+		(property "Sim.Pins" "1=K 2=A"
+			(at 731.52 92.71 0)
+			(hide yes)
 			(show_name no)
 			(do_not_autoplace no)
@@
 	)
 	(symbol
-		(lib_id "PAL-snes-1chip-schematic-rescue:D_Small_ALT-Device")
+		(lib_id "Device:D_Small")
 		(at 721.36 92.71 0)
 		(unit 1)
@@
 			)
 		)
-		(property "Description" ""
+		(property "Description" "Diode, small symbol"
+			(at 721.36 92.71 0)
+			(hide yes)
+			(show_name no)
+			(do_not_autoplace no)
+			(effects
+				(font
+					(size 1.27 1.27)
+				)
+			)
+		)
+		(property "Sim.Device" "D"
 			(at 721.36 92.71 0)
+			(hide yes)
+			(show_name no)
+			(do_not_autoplace no)
+			(effects
+				(font
+					(size 1.27 1.27)
+				)
+			)
+		)
+		(property "Sim.Pins" "1=K 2=A"
+			(at 721.36 92.71 0)
+			(hide yes)
 			(show_name no)
 			(do_not_autoplace no)
@@
 	)
 	(symbol
-		(lib_id "SNES_parts:RF_MODULATOR")
+		(lib_id "SNES_Library:RFMODULATOR")
 		(at 588.01 229.87 0)
 		(unit 1)
@@
 		)
 		(property "Footprint" "SNES_Library:RFModulator"
-			(at 588.01 237.49 0)
+			(at 582.93 226.06 0)
 			(hide yes)
 			(show_name no)
@@
 			(effects
 				(font
-					(size 1.524 1.524)
+					(size 1.27 1.27)
 				)
 			)
 		)
 		(property "Datasheet" ""
-			(at 588.01 237.49 0)
+			(at 582.93 226.06 0)
 			(hide yes)
 			(show_name no)
@@
 			(effects
 				(font
-					(size 1.524 1.524)
+					(size 1.27 1.27)
 				)
 			)
@@
 		(property "Description" ""
 			(at 588.01 229.87 0)
+			(hide yes)
 			(show_name no)
 			(do_not_autoplace no)
@@
 	(symbol
 		(lib_id "Device:D_Zener_Dual_CommonCathode_AAK")
-		(at 589.915 35.56 180)
+		(at 590.55 35.56 180)
 		(unit 1)
 		(body_style 1)
@@
 		(fields_autoplaced yes)
 		(property "Reference" "D1"
-			(at 589.915 39.37 0)
+			(at 590.55 39.37 0)
 			(show_name no)
 			(do_not_autoplace no)
@@
 		)
 		(property "Value" "12V Zener"
-			(at 589.915 41.91 0)
+			(at 590.55 41.91 0)
 			(show_name no)
 			(do_not_autoplace no)
@@
 		)
 		(property "Footprint" "Package_TO_SOT_SMD:SC-59"
-			(at 589.915 35.56 0)
+			(at 590.55 35.56 0)
 			(hide yes)
 			(show_name no)
@@
 		)
 		(property "Datasheet" ""
-			(at 589.915 35.56 0)
+			(at 590.55 35.56 0)
 			(hide yes)
 			(show_name no)
@@
 		)
 		(property "Description" ""
-			(at 589.915 35.56 0)
+			(at 590.55 35.56 0)
 			(hide yes)
 			(show_name no)
